Commit message: 修复躯干碰撞体接地导致四个车轮悬空
用 gz sdf -p 逐个计算碰撞体最低点发现，躯干底座的碰撞圆柱体
(origin z=-0.05, length=0.1) 在模型系里最低点是 -0.0638，而四个
车轮球体最低点是 -0.0655，两者只差 1.7mm。整机 39kg 几乎全部
压在这个"躯干肚皮"上，车轮承担的法向力 N≈0，摩擦力 F=mu*N≈0。

直接证据：实测静止高度 z=0.1342 正好等于"肚皮坐地"算出的高度，
而不是"车轮坐地"的高度；把 mu 从 0.7 拉到 5.0 车身照样不动，
说明和摩擦系数完全无关。

把圆柱体上移到 z=-0.01，让四个车轮成为唯一接地点，同时保留躯干
碰撞体积（撞货架、碰撞诱发倾倒的研究还需要它）。上移后车轮比
肚皮低约 42mm 净空。

这条同时改写了历史结论：第一轮记录的"各向异性摩擦在小轮子上失效"、
以及后来"必须用 VelocityControl 绕开摩擦"的判断，很可能一直都是被
这个肚皮接地问题误导的——不是 DART 摩擦数值不稳定，是车轮根本没受力。

Co-Authored-By: Claude <noreply@anthropic.com>

File: ws_robot/src/astribot_s1_description/urdf/astribot_s1_torso_wheel.xacro (robot description, xacro)
@@ -38,5 +38,21 @@
     </visual>
     <collision>
-      <origin rpy="0 0 0" xyz="0 0 -0.05"/>
+      <!-- !!! 实测踩坑记录（力控重构方案，"轮子转但车身完全不动"的真正根因）!!!：
+           这个碰撞圆柱体原来是 origin z=-0.05 + length=0.1，也就是在 torso_base 系里
+           从 z=-0.10 一直伸到 z=0.0。实测用 gz sdf -p 逐个算碰撞体最低点发现：
+             轮子球体最低点(模型系) = -0.0655
+             这个圆柱体最低点(模型系) = -0.0638
+           **两者只差 1.7mm** ——也就是说整机 39kg 的重量几乎全压在这个"躯干肚皮"
+           圆柱体上，四个轮子只比它低 1.7mm、几乎不承担法向力(N≈0)，
+           摩擦力 F=mu*N≈0 —— 轮子空转、车身一动不动，而且**跟 mu 配多大完全无关**
+           (实测把 mu 从 0.7 拉到 5.0 也不动)。实测静止高度 z=0.1342 正好等于
+           "肚皮坐在地上"算出来的高度，不是"轮子坐在地上"的高度，是直接证据。
+           这条同时改写了历史结论：第一轮"各向异性摩擦在小轮子上失效"、
+           以及后来"必须用 VelocityControl 绕开摩擦"的判断，很可能一直都是被
+           这个肚皮接地问题误导的——不是 DART 摩擦数值不稳定，是轮子根本没受力。
+           修法：把圆柱体上移，让四个轮子成为唯一接地点，同时保留一个躯干碰撞
+           体积(撞货架/碰撞诱发倾倒研究还需要它)。上移 0.04m 后轮子比肚皮低
+           约 42mm 净空，够用且不夸张。 -->
+      <origin rpy="0 0 0" xyz="0 0 -0.01"/>
       <geometry>
         <cylinder length="0.1" radius="0.3"/>
