Commit message: Gate 1(部分)：关节限位切到厂商 per-part 模型 + 一致性测试 + 修好探针这台仪器
--- 限位切换 ---

真值源改为各部件 yaml 的 model: 字段指向的 per-part 文件（SDK 运行时真正加载
的那一份），不再用 astribot_whole_body_with_wheel.urdf。

先确认了切换的范围：per-part 与 whole_body 在**关节原点与惯量/质量上逐项完全
一致（0 处差异）**，只有限位表不同。所以只需换限位，几何与惯量一行都不用动。
这也解释了为什么不能直接 xacro:include 厂商 URDF——per-part 文件完全无 mesh，
且同样缺 base_link/link_1/link_2/link_6 的 collision。

臂（两侧）：
  joint_1 -3.0~3.0 -> -3.1~3.1        joint_2 -1.4~0.4 -> -1.53~0.46
  joint_3 左-3.0~1.4/右-1.4~3.1 -> 两侧统一 ±3.1
  joint_4  0.0~2.4 -> -0.06~2.61      joint_5 ±2.0 v15 -> ±2.56 v20
  joint_6 ±0.6 -> ±0.76               joint_7 ±1.4 -> ±1.53
躯干（**安全相关**）：四个关节速度 6.0 -> 1.8 rad/s；joint_4 ±1.5 -> ±1.2。
  原先比真机控制栈认定的 1.8 宽 3.3 倍，时间最优参数化跑满时躯干段速度可达
  真机限位 3 倍，而 Gazebo 会照 URDF 老实执行、什么都不报。收紧后节拍变长，
  这是正确的代价。
头部两关节各版本一致，未动。

两个副作用已在注释里写明：joint_3 放开后可能进入原先被限位挡住的自碰撞区域
（碰撞由 CollisionValidator 实际校验，不靠限位兜底）；joint_4 下限 -0.06 允许
略微越过"肘部完全伸直"这个精确奇异构型，故奇异点监视器不能关。

--- 一致性测试（已验证非空跑）---

新增 test/test_joint_limits_parity.py：展开本包 xacro 与 per-part 模型逐项比对
限位与关节原点，另有一个哨兵测试专挡"退回 whole_body 特征值"这个具体历史错误。
故意把躯干速度改回 6.0 验证过：2 个测试失败且报错直接点出根因，不是空跑。

--- 修正一处方法学错误：探针指标此前是随机的 ---

方案文档里把"可用候选数明显增加"写成 Gate 1 验收标准，但从没量过这个指标的
噪声底。实测同一份配置连跑三次得到 48/80、46/80、47/80——run-to-round 抖动 ±2，
与要观测的效果同量级。拿噪声当信号，判据本身不成立。
（连带说明早先写进 README 的"80 个候选 50 个可用"是个软数字。）

根因：probeTcpPose 只调一次 setFromIK，且沿用闭链那套 ik_timeout 0.01s。
setFromIK 是随机重启局部解算器，小预算下结果本就随机。

修法不是调参凑数，而是改语义：新增 demo.transport_probe_ik_timeout(0.05) 与
transport_probe_ik_attempts(20)，重试至"任一次拿到合法解"即判可达——
点估计换成稳定下界。探针不在控制环里，慢无所谓。

修好后两次独立运行都是 54/80，完全一致；抖动消失。
可用候选 47±2 -> 54（限位放宽确实有效，但只有压掉噪声才看得出来）。
IK 无解稳定在 23 个：提高预算没有减少它，说明这 23 个是真不可达而非超时假象——
比原来"23~26 浮动"硬得多。

--- 尚未做（Gate 1 剩余）---
TCP link（法兰 -y 0.15）、夹爪（6 物理关节 + 1 抽象关节 0~100）、
SRDF 的 end_effector/gripper 组。

File: ws_robot/src/astribot_s1_description/urdf/astribot_s1_arm.xacro (robot description, xacro)
@@ -6,7 +6,34 @@
   上下限 两侧不同，因此把这些差异值做成宏参数，其余数值直接写死在宏体内，
   避免用符号翻转公式去"推导"左右差异（原始工程数据不是简单镜像关系，直接照抄原文件数值最安全）。
-  数值来源：astribot_config/robot_config/astribot_s1/model/astribot_whole_body_with_wheel.urdf
-  （未改动任何数值），只修正了 mesh 路径，并为缺失 collision 的 link
-  （base_link、link_1、link_2、link_6）按 STL 包围盒补了简化碰撞体。
+  数值来源（2026-08-20 改）：关节限位以
+  astribot_config/robot_config/astribot_s1/model/astribot_arm_left.urdf
+  与 astribot_arm_right.urdf（**per-part 模型**）为准。
+  连杆惯量/质量/关节原点仍取自 astribot_whole_body_with_wheel.urdf ——
+  实测这两份在惯量与关节原点上**逐项完全一致**（0 处差异），只有限位表不同，
+  所以只需要换限位，不需要动几何与惯量。
+  mesh 路径为本工程修正；为缺失 collision 的 link（base_link、link_1、link_2、link_6）
+  按 STL 包围盒补了简化碰撞体 —— per-part 模型同样缺这几个 collision 且完全无 mesh，
+  这也正是不能直接 xacro:include 厂商 URDF 的原因。
+  !!! 为什么换成 per-part：厂商 ship 了四份互不一致的模型 !!!
+  各部件 yaml 的 model: 字段指向的才是 SDK 运行时真正加载的那一份，
+  whole_body_*.urdf 一份都没被引用。以 SDK 加载的为准才能与真机对齐。
+  详见 docs/sim_real_alignment.md 第 0 节。
+  本次限位变更（旧 = whole_body_with_wheel，新 = per-part）：
+    joint_1  -3.0~3.0        -> -3.1~3.1
+    joint_2  -1.4~0.4        -> -1.53~0.46
+    joint_3  左 -3.0~1.4 / 右 -1.4~3.1  -> 两侧统一 -3.1~3.1
+    joint_4   0.0~2.4        -> -0.06~2.61
+    joint_5  -2.0~2.0 v15    -> -2.56~2.56 v20
+    joint_6  -0.6~0.6        -> -0.76~0.76
+    joint_7  -1.4~1.4        -> -1.53~1.53
+  注意两点副作用：
+  1) joint_3 原先左右不对称（镜像限制），per-band 模型两侧都是 ±3.1，
+     故 joint3_lower/joint3_upper 这对参数现在两侧取值相同。参数保留不删 ——
+     它记录了这个非对称限制曾经存在，且换机型时仍是有用的钩子。
+     放开后搜索空间变大，可能进入原先被限位挡住的自碰撞区域，
+     但碰撞由 CollisionValidator 实际校验，不靠限位兜底。
+  2) joint_4 下限从 0.0 放到 -0.06，意味着允许略微越过"肘部完全伸直"这个
+     精确奇异构型（实测 joint_4=0 时 sigma_min=0.0077）。真机允许，所以照抄，
+     但这让奇异点监视器变得更重要，不要关掉它。
 -->
 <robot xmlns:xacro="http://www.ros.org/wiki/xacro">
@@ -72,5 +99,5 @@
       <child link="astribot_arm_${side}_link_1"/>
       <axis xyz="0 0 1"/>
-      <limit effort="265" lower="-3.0" upper="3.0" velocity="8.4"/>
+      <limit effort="265" lower="-3.1" upper="3.1" velocity="8.4"/>
     </joint>
     <!-- ===== link_2：左右 mesh/惯量不同（肩部结构件） ===== -->
@@ -104,5 +131,5 @@
       <child link="astribot_arm_${side}_link_2"/>
       <axis xyz="0 0 1"/>
-      <limit effort="265" lower="-1.4" upper="0.4" velocity="8.4"/>
+      <limit effort="265" lower="-1.53" upper="0.46" velocity="8.4"/>
     </joint>
     <!-- ===== link_3：两侧惯量相同，但 joint_3 上下限左右相反（镜像安装），已作为参数传入 ===== -->
@@ -163,5 +190,5 @@
       <child link="astribot_arm_${side}_link_4"/>
       <axis xyz="0 0 1"/>
-      <limit effort="142" lower="0.0" upper="2.4" velocity="15"/>
+      <limit effort="142" lower="-0.06" upper="2.61" velocity="15"/>
     </joint>
     <link name="astribot_arm_${side}_link_5">
@@ -192,5 +219,5 @@
       <child link="astribot_arm_${side}_link_5"/>
       <axis xyz="0 0 1"/>
-      <limit effort="71" lower="-2.0" upper="2.0" velocity="15"/>
+      <limit effort="71" lower="-2.56" upper="2.56" velocity="20"/>
     </joint>
     <link name="astribot_arm_${side}_link_6">
@@ -222,5 +249,5 @@
       <child link="astribot_arm_${side}_link_6"/>
       <axis xyz="0 0 1"/>
-      <limit effort="20" lower="-0.6" upper="0.6" velocity="16.8"/>
+      <limit effort="20" lower="-0.76" upper="0.76" velocity="16.8"/>
     </joint>
     <link name="astribot_arm_${side}_link_7">
@@ -251,5 +278,5 @@
       <child link="astribot_arm_${side}_link_7"/>
       <axis xyz="0 0 1"/>
-      <limit effort="20" lower="-1.4" upper="1.4" velocity="16.8"/>
+      <limit effort="20" lower="-1.53" upper="1.53" velocity="16.8"/>
     </joint>
     <!-- 末端工具挂载点（法兰），预留给夹爪/工具，本方案未挂夹爪，保留 fixed link 便于后续扩展 -->
@@ -286,5 +313,5 @@
     link2_ixx="0.00360751" link2_ixy="-0.00009193" link2_ixz="0.00007764"
     link2_iyy="0.00283747" link2_iyz="0.00054945" link2_izz="0.00172927"
-    joint3_lower="-3.0" joint3_upper="1.4"
+    joint3_lower="-3.1" joint3_upper="3.1"
     base_fixed_rpy="0 -1.22173 -1.5707963" base_fixed_xyz="0 0.06449 0.02348"/>
   <!-- ================= 右臂实例化（数值取自原 URDF astribot_arm_right_* 数据） ================= -->
@@ -301,5 +328,5 @@
     link2_ixx="0.00394196" link2_ixy="-8.846e-05" link2_ixz="-3.742e-05"
     link2_iyy="0.00316298" link2_iyz="-0.0007079" link2_izz="0.00177295"
-    joint3_lower="-1.4" joint3_upper="3.1"
+    joint3_lower="-3.1" joint3_upper="3.1"
     base_fixed_rpy="0 -1.22173 1.5707963" base_fixed_xyz="0 -0.06449 0.02348"/>
 </robot>

File: ws_robot/src/astribot_s1_description/urdf/astribot_s1_torso_wheel.xacro (robot description, xacro)
@@ -237,4 +237,19 @@
     </collision>
   </link>
+  <!-- ===== 躯干 4 自由度 =====
+       !!! 限位以 per-part 模型 model/astribot_torso.urdf 为准（2026-08-20 改）!!!
+       各部件 yaml 的 model: 字段指向的才是 SDK 运行时加载的那一份；
+       whole_body_*.urdf 一份都没被引用。详见 docs/sim_real_alignment.md 第 0 节。
+       本次变更里**速度限位是安全相关的**，不是可选优化：
+         joint_1  0.0~1.4  v6.0  ->  -0.04~1.5  v1.8
+         joint_2 -2.3~0.0  v6.0  ->  -2.3~0.06  v1.8
+         joint_3  0.0~2.3  v6.0  ->  -0.4~2.3   v1.8
+         joint_4 -1.5~1.5  v6.0  ->  -1.2~1.2   v1.8
+       原先 6.0 rad/s 比真机控制栈认定的 1.8 rad/s 宽 3.3 倍 ——
+       也就是说 optimized_velocity_scaling: 0.90 跑满的"时间最优"轨迹，
+       躯干段速度可以达到真机限位的 3 倍，而 Gazebo 会照 URDF 老实执行、
+       什么都不报。收紧后节拍会相应变长，这是正确的代价。
+       joint_4 位置范围同样收窄（±1.5 -> ±1.2），方向也是变安全。
+  -->
   <joint name="astribot_torso_joint_1" type="revolute">
     <origin rpy="-1.5708 1.5708 0" xyz="0 0 0.12"/>
@@ -242,5 +257,5 @@
     <child link="astribot_torso_link_1"/>
     <axis xyz="0 0 1"/>
-    <limit effort="100" lower="0.0" upper="1.4" velocity="6.0"/>
+    <limit effort="100" lower="-0.04" upper="1.5" velocity="1.8"/>
   </joint>
   <link name="astribot_torso_link_2">
@@ -271,5 +286,5 @@
     <child link="astribot_torso_link_2"/>
     <axis xyz="0 0 1"/>
-    <limit effort="100" lower="-2.3" upper="0.0" velocity="6.0"/>
+    <limit effort="100" lower="-2.3" upper="0.06" velocity="1.8"/>
   </joint>
   <link name="astribot_torso_link_3">
@@ -300,5 +315,5 @@
     <child link="astribot_torso_link_3"/>
     <axis xyz="0 0 1"/>
-    <limit effort="100" lower="0.0" upper="2.3" velocity="6.0"/>
+    <limit effort="100" lower="-0.4" upper="2.3" velocity="1.8"/>
   </joint>
   <link name="astribot_torso_link_4">
@@ -331,5 +346,5 @@
     <child link="astribot_torso_link_4"/>
     <axis xyz="0 0 1"/>
-    <limit effort="100" lower="-1.5" upper="1.5" velocity="6.0"/>
+    <limit effort="100" lower="-1.2" upper="1.2" velocity="1.8"/>
   </joint>
   <!-- 质量/惯量为 0 的虚拟挂载点，双臂与头部都挂在这里 -->
