Commit message: Gate 1 全栈验证（Gazebo+RViz+执行）：σ 疑问查清，并测出 Gazebo mimic 有 7.8° 稳态误差
--- 1. 上一轮那个"σ=0.0077 却 PASS"查清了，推测成立 ---
execute:=true 实跑后六步最差 σ 变成
0.1156/0.1377/0.1380/0.1653/0.1658/0.1570，全程最差 0.1156 = 阈值的 5.8 倍。
0.0077 确实是**起始状态**带进来的：execute:=false 时机器人从不移动，
六步全从同一个零位(joint_4=0 肘部完全伸直)重新起步；真执行后每步从上一步终点起步。
奇异监视器从来没失效 —— 它报的是那条真的起于奇异位形的轨迹的最差值。

--- 2. 全栈验证结果 ---
· gripper_left/right_controller 均 Configured and activated
· /joint_states 26 个关节，含两个夹爪主动关节（5 个 mimic 正确地不在其中）
· 下发 0.93 rad -> 主动关节到位 0.93000，action SUCCEEDED
· transport execute:=true **6/6 SUCCESS**，无 deviates/Invalid Trajectory/ABORTED
  （早先加的 waitUntilSettled 在真执行下站住了）
· 末端落点 TF 实测 (0.170,0.276,0.929) 与第6步目标逐位一致，
  姿态 (0.707,0,0,0.707) = 本轮推导出的俯视抓取姿态
· 节拍 1.583s（不执行时 3.525s，因为每步不再从零位长距离起步）

--- 3. 新测出的 sim/plan 差异：Gazebo mimic 有 7.8° 稳态误差 ---
此前记为"未实测"。给主动关节下发 0.93 rad 后，把 Gazebo 内部连杆位姿
(ign topic /world/default/pose/info) 与 TF(RSP 按 mimic 算的)逐个比：
  Link_L11  差 0.21 mm  —— 父关节是主动关节 L1，一致
  Link_R11  差 7.47 mm  —— 父关节 R1 是 mimic 关节，不一致
用 R11 实测位置反解 R1(Gazebo)=0.7940 rad，mimic 应给 0.9300 rad，差 -7.79°
(残差 0.21 mm)。0.794 既不是 0(那会差 42.5 mm)也不像自由摆动的随机值，
所以 gz_ros2_control 确实在执行 mimic，只是像个带稳态误差的软约束。

影响范围：MoveIt 侧 mimic 精确，规划与碰撞不受影响；Gazebo 侧右指比 MoveIt
认为的少闭合约 15%。当前 transport 没有夹取/attach 动作、不依赖 Gazebo 接触物理，
所以不进入结论 —— 但做夹持力/接触实验前必须先解决。

Co-Authored-By: Claude <noreply@anthropic.com>

File: ws_robot/src/astribot_s1_description/urdf/astribot_s1_gripper.xacro (robot description, xacro)
@@ -127,10 +127,26 @@
   代价必须知道：**Gazebo 里这 6 个连杆的转动惯量被高估约 30 倍**，如果以后要在
   Gazebo 里做夹爪动力学（抓取力、指尖接触），这个值不能用。当前不用，故不改。
+  ================== Gazebo 侧 mimic：已实测，有 7.8° 稳态误差 ==================
+  此前这里写的是"Humble 的 gz_ros2_control 对 URDF <mimic> 的支持情况未实测，
+  从动关节可能受重力自由摆动"。**已实测（2026-08-20），结论是支持但不精确。**
+  测法：接 Gazebo 起全栈，给主动关节 joint_L1 下发 0.93 rad 并确认到位，
+  然后拿 Gazebo 内部的连杆位姿（ign topic /world/default/pose/info）
+  与 TF（robot_state_publisher 按 mimic 算出来的）逐个比。
+    astribot_gripper_left_Link_L11   Gazebo 与 TF 差 0.21 mm  —— 一致
+    astribot_gripper_left_Link_R11   Gazebo 与 TF 差 7.47 mm  —— 不一致
+  L11 的父关节是主动关节 L1（Gazebo 里真的被驱动），所以一致；
+  R11 的父关节 R1 是 mimic 关节。用 R11 的实测位置反解 R1 的真实角度：
+    R1(Gazebo) = 0.7940 rad，而 mimic 应给 0.9300 rad，
+    差 -0.1360 rad = **-7.79°**（反解残差 0.21 mm，解是干净的）。
+  注意 0.794 既不是 0（那会差 42.5 mm）也不是自由摆动的随机值 ——
+  所以 gz_ros2_control 确实在执行 mimic，只是像个有限刚度/带稳态误差的约束。
+  影响范围要分清：
+    · MoveIt 侧（规划与碰撞）用自己的 RobotState，mimic 是精确的，与厂商模型一致 ——
+      **规划结果不受影响**。
+    · Gazebo 侧的右指比 MoveIt 认为的少闭合约 15%。只要不依赖 Gazebo 的接触物理
+      做抓取（当前 transport 场景没有夹取/attach 动作），这个差异不进入结论。
+    · 一旦要用 Gazebo 做夹持力/接触实验，这 7.8° 必须先解决，
+      否则两指不对称、接触点也不对。
   ================== 本阶段（模型对齐）不做什么 ==================
-  · 不给夹爪配 Gazebo 侧的 mimic 执行。Humble 的 gz_ros2_control 对 URDF
-    <mimic> 的支持情况未实测，从动关节可能在 Gazebo 里受重力自由摆动。
-    本阶段目标是 MoveIt 的运动学/碰撞模型与厂商一致，mimic 在 MoveIt 侧
-    是可靠的（从动关节不计入活动自由度）。Gazebo 侧的表现留到需要时实测再定，
-    不在这里凭猜测加补丁。
   · 不做夹持力。厂商的夹持力是另一条接口（set_effector_max_force，10~80 N，
     随机器人模式变化），不是关节 effort 限位。URDF 里的 effort 沿用源里的 1.0
