Commit message: Gate 1 完成：夹爪建成真实关节 + TCP 改到 tcp_link + 修好两台仪器
夹爪缺失的真正代价不在"不能抓"，在**碰撞模型缺了一大块**：
厂商自己的碰撞模型(whole_body.sdf 的 link_7)用 opened_gripper.obj，
换算到 link_7 系覆盖 y∈[-0.1997,-0.048]、x 宽 0.148；
本仓库此前只有一个 sphere r=0.05(y∈[-0.05,0.05])。
即沿抓取方向少 0.15m、横向少 0.148m，整个夹爪不在碰撞模型里 ——
规划出的轨迹会用夹爪去撞东西，而仿真里一切正常。

--- 做了什么 ---
· 新增 astribot_s1_gripper.xacro：每侧 7 link / 6 关节
  (joint_L1 主动 0~0.93rad，5 个 mimic 比例 ±1)。
  几何/轴向/行程/耦合取 MJCF，碰撞 mesh 与基座装法取 whole_body_with_gripper.sdf。
  平行四边形机构使 URDF mimic 在这里是**精确**表达而非近似。
· tool_link 改纯坐标系 + 新增 tcp_link(法兰 -y 0.15，厂商 effector_to_tool_pose)；
  SRDF 各组 tip 与 manipulation 的 TCP 全部指过去。
· SRDF：gripper_left/right 组 + end_effector + open/closed 状态 + 夹爪 10 对碰撞关闭。
· 控制链路一次配齐：ros2_control / joint_state_broadcaster 白名单 /
  两个 gripper_*_controller / moveit_controllers / joint_limits / launch spawner。
  漏任一处 move_group 报 Missing ..._joint_L1 且**整个规划功能不可用**。
· test_gripper_model.py 27 条，注入故障验证过非空跑。

--- 修好的两台仪器（都曾给出假结论）---
1. transport_probe：原判据"可用候选应明显增加"是拿噪声当信号 ——
   同配置连跑三次 48/46/47(±2 抖动，与效果同量级)。改语义为
   50ms×20 次取稳定下界后，复测 54/54 一致，IK 无解稳定在 23。
2. test_gripper_model 的平行夹爪不变量：最初把 mimic 比例写死在测试里，
   注入 ratio=-1 故障照样通过 —— 验证的是我的假设不是模型。改成从 URDF 读。
   质量守恒判据同理：原来拿整机质量做分母，注入"法兰惯量没清零"只有 1.664%
   (单侧更只有 0.83%，会从 1% 门槛下溜过)；改成比腕部子树后同故障是 84.3%。
3. self_collision_pair_generator：max_contacts 写死 200，而加夹爪后对数
   465→820。改成按 link 数现算。

--- 发现的厂商不一致（已记进注释并被测试钉住）---
· L11/R11 销轴两源差 7.0mm(MJCF vs SDF) => 指尖沿抓取方向有 7mm 不确定度。
· 碰撞 mesh 不是精确镜像，是各自独立简化(L11 139面 vs R11 122面)，
  而运动学侧严格镜像(实测差 0.000000)。销轴处"刚好擦到"两侧判定不同：
  L11<->L2 9.32% vs R11<->R2 100%。这是 SRDF 里唯一一处按机构而非按采样
  统计关掉的碰撞对(销轴物理上永远接触，不关会废掉约 9% 夹爪区间)。
  排查中错怪过预压角不一致和 max_contacts 截断，两次改动都没改变结果。

--- 尚未做 ---
· 重跑 transport_probe 定新的 A/B 与 grasp_z_offset：旧的抓取余量数字
  全部作废(方法有效、数字不可信)。σ 只取决于手臂 7 关节，不受影响。
· transport 场景还没有"张开/闭合 + attach 物体"动作，物体仍不跟着走。
· Gazebo 侧 mimic 执行未实测(Humble 的 gz_ros2_control 支持情况未知)。
· 夹爪 6 连杆惯量是厂商占位值(0.03kg 配 I=0.001 => 回转半径 0.18m，物理上
  不可能)，照抄并标出；Gazebo 里做夹爪动力学前必须标定。

Co-Authored-By: Claude <noreply@anthropic.com>

File: ws_robot/src/astribot_s1_description/urdf/astribot_s1.xacro (robot description, xacro)
@@ -15,4 +15,15 @@
   <xacro:arg name="use_lidar" default="true"/>
   <xacro:arg name="use_camera" default="true"/>
+  <!-- use_gripper：是否把平行夹爪作为真实关节模块建模。
+       true（默认，与真机一致）：加载 astribot_s1_gripper.xacro，两臂末端各挂
+         7 个 link / 6 个关节（1 主动 + 5 mimic），法兰 tool_link 的集中惯量清零。
+       false：夹爪不建模，退回厂商 per-part 模型的表示法（0.64763 kg 集中惯量
+         挂在法兰上，腕部碰撞只有 link_7 的 sphere r=0.05）。
+       !!! 不要为了"让规划快一点"而随手关掉它 !!!
+       关掉后腕部碰撞体沿抓取方向少 0.15 m、横向少 0.148 m，夹爪整体不在碰撞
+       模型里 —— 规划出来的轨迹在真机上会用夹爪去撞东西。这个开关存在的意义是
+       "与厂商那份集中惯量模型做对照实验"，不是性能旋钮。
+       详见 astribot_s1_gripper.xacro 文件头。 -->
+  <xacro:arg name="use_gripper" default="true"/>
   <!-- 双 Livox Mid-360 安装位姿：左前 + 右后对角布局（用户指定），扩大合并视场、
        减少互相遮挡的盲区（默认值，可外部覆盖）。
@@ -50,11 +61,26 @@
   <xacro:property name="use_camera_prop" value="$(arg use_camera)"/>
   <xacro:property name="robot_name_prop" value="$(arg robot_name)"/>
+  <!-- use_gripper 必须在 include 之前定义成 property：astribot_s1_arm.xacro 在它
+       自己文件末尾就地实例化左右两条臂，宏体里用 ${use_gripper} 决定法兰惯量的
+       归属（见该文件 tool_link 处）。property 在 include 之前定义，被包含的文件
+       才看得到。这里刻意不在 arm xacro 里重复声明同名 xacro:arg —— 同一个 arg
+       声明两次的行为在各版本 xacro 里并不一致，只留一处声明最稳。 -->
+  <xacro:property name="use_gripper" value="$(arg use_gripper)"/>
   <!-- ============ 载入各功能模块 ============ -->
   <xacro:include filename="$(find astribot_s1_description)/urdf/astribot_s1_torso_wheel.xacro"/>
   <xacro:include filename="$(find astribot_s1_description)/urdf/astribot_s1_head.xacro"/>
   <xacro:include filename="$(find astribot_s1_description)/urdf/astribot_s1_arm.xacro"/>
+  <xacro:include filename="$(find astribot_s1_description)/urdf/astribot_s1_gripper.xacro"/>
   <xacro:include filename="$(find astribot_s1_description)/urdf/astribot_s1_sensors.xacro"/>
   <xacro:include filename="$(find astribot_s1_description)/urdf/astribot_s1_ros2_control.xacro"/>
   <xacro:include filename="$(find astribot_s1_description)/urdf/astribot_s1.gazebo.xacro"/>
+  <!-- ============ 平行夹爪（左右各一具，挂在各自 link_7 上） ============
+       夹爪相对法兰的装法左右完全相同（实测厂商 MJCF 左右两份模型除一处命名笔误
+       外数值一处不差，SDF 侧左右 6 个关节 pose/axis 也逐项相同），所以同一个宏
+       实例化两次、不做镜像取反。 -->
+  <xacro:if value="${use_gripper}">
+    <xacro:astribot_s1_gripper side="left"  parent="astribot_arm_left_link_7"/>
+    <xacro:astribot_s1_gripper side="right" parent="astribot_arm_right_link_7"/>
+  </xacro:if>
   <!-- ============ 传感器（按参数开关，默认都打开） ============ -->
   <!-- 双 Livox Mid-360：分别实例化 left/right，frame_id 各自独立

File: ws_robot/src/astribot_s1_description/urdf/astribot_s1_arm.xacro (robot description, xacro)
@@ -280,11 +280,45 @@
       <limit effort="20" lower="-1.53" upper="1.53" velocity="16.8"/>
     </joint>
-    <!-- 末端工具挂载点（法兰），预留给夹爪/工具，本方案未挂夹爪，保留 fixed link 便于后续扩展 -->
+    <!-- ===== 末端：法兰(tool_link) -> TCP(tcp_link) =====
+         !!! tool_link 不是 TCP，这是本次改动纠正的一个实质错误 !!!
+         tool_link 与 link_7 的 origin 完全重合（xyz 0 0 0），也就是说它就是**法兰面**。
+         之前把它当笛卡尔目标用，等价于"让法兰去到目标点"，而真正该到位的是
+         两指之间的夹持点 —— 两者相差 0.15 m。而且法兰正好坐在腕部碰撞体里，
+         导致"TCP 贴着物体"必然报碰撞（这条坑已单独记录过）。
+         TCP 偏置来源（厂商配置，不是我估的）：
+           astribot_config/robot_config/astribot_s1/astribot_arm_left.yaml
+             effector_to_tool_pose: [0.0, -0.15, 0.0,  0.0, 0.0, 0.0, 1.0]
+         即位置 (0, -0.15, 0)、姿态四元数 (0,0,0,1) = 不旋转。右臂 yaml 同值。
+         为什么是 -y 而不是别的方向：夹爪基座以 rpy(1.5708,0,0) 装在 link_7 上，
+         把基座的 +z（张合机构伸出方向）转到了 link_7 的 -y。见 astribot_s1_gripper.xacro。
+         0.15 这个数的独立几何佐证（不是只信 yaml 一处）：
+         按 MJCF 算指尖胶垫中心在基座系 z ≈ 0.0511+0.0364+0.036 = 0.1235，
+         基座原点在 link_7 系 y ≈ -0.0506，故胶垫中心在 link_7 系 y ≈ -0.174，
+         胶垫半高 0.03 => 胶垫沿 y 覆盖 [-0.144, -0.204]。
+         TCP 的 -0.15 正落在胶垫的近端 —— 是"指根附近的夹持参考点"，位置合理。
+         同时它落在 link_7 的 sphere r=0.05（覆盖 y ∈ [-0.05, 0.05]）之外、
+         也在夹爪基座碰撞 mesh（覆盖 y ∈ [-0.1376, -0.048]）之外，
+         张开时两指分开约 105 mm、指间是空的 —— 所以 TCP 处不再自带碰撞。 -->
     <link name="astribot_arm_${side}_tool_link">
-      <inertial>
-        <origin rpy="0 0 0" xyz="-0.00019766 -0.10719761 0.00190898"/>
-        <mass value="0.64762850"/>
-        <inertia ixx="0.00152446" ixy="0.00000144" ixz="-0.00000058" iyy="0.00033076" iyz="0.00004144" izz="0.00156453"/>
-      </inertial>
+      <!-- 法兰上那 0.64763 kg 集中惯量的归属，取决于夹爪是否作为独立模块建模：
+           use_gripper=false（厂商 per-part / whole_body 模型的表示法）：
+             夹爪不建模，它的质量以集中惯量的形式挂在法兰上。质心在 -y 0.107，
+             正是夹爪整体质心的位置。这是照抄厂商 per-part 模型的原值。
+           use_gripper=true（本工程默认，见 astribot_s1_gripper.xacro）：
+             夹爪已经是 7 个真实 link（基座 0.4 + 6 指连杆 0.254 = 0.654 kg），
+             法兰这里**必须清零**，否则夹爪质量被算两遍。
+             清零后总质量 0.12772019(link_7) + 0.654 = 0.78172，
+             对比清零前 0.12772019 + 0.64762850 = 0.77535，差 +0.0064 kg(+0.82%)。
+             这 0.82% 不是我引入的误差，是厂商"集中表示"与"分体表示"两份模型
+             本来就有的差异（whole_body.sdf 的 link_7 集中质量 0.775349
+             对 whole_body_with_gripper.sdf 的 0.527722+0.254=0.781722）。
+             test_gripper_model.py 按 1% 断言这条，差异变大会被测出来。 -->
+      <xacro:unless value="${use_gripper}">
+        <inertial>
+          <origin rpy="0 0 0" xyz="-0.00019766 -0.10719761 0.00190898"/>
+          <mass value="0.64762850"/>
+          <inertia ixx="0.00152446" ixy="0.00000144" ixz="-0.00000058" iyy="0.00033076" iyz="0.00004144" izz="0.00156453"/>
+        </inertial>
+      </xacro:unless>
     </link>
     <joint name="astribot_arm_${side}_tool_joint" type="fixed">
@@ -292,4 +326,13 @@
       <parent link="astribot_arm_${side}_link_7"/>
       <child link="astribot_arm_${side}_tool_link"/>
+    </joint>
+    <!-- TCP：纯坐标系，无 visual/无 collision/无惯量。
+         无碰撞几何是刻意的 —— 它是 IK 与笛卡尔约束的参考系，不该自己制造碰撞。
+         SRDF 各规划组的 tip 与 manipulation_params.yaml 的 TCP 都指向这里。 -->
+    <link name="astribot_arm_${side}_tcp_link"/>
+    <joint name="astribot_arm_${side}_tcp_joint" type="fixed">
+      <origin rpy="0 0 0" xyz="0 -0.15 0"/>
+      <parent link="astribot_arm_${side}_tool_link"/>
+      <child link="astribot_arm_${side}_tcp_link"/>
     </joint>
     <!-- 挂到躯干末端虚拟点，左右各自的安装角度/偏移不同 -->

File: ws_robot/src/astribot_s1_description/urdf/astribot_s1_ros2_control.xacro (robot description, xacro)
@@ -82,4 +82,19 @@
       <xacro:astribot_s1_effort_wheel_joint name="wheel_RR_Joint"/>
       <xacro:astribot_s1_effort_wheel_joint name="wheel_LR_Joint"/>
+      <!-- 夹爪：每侧只声明**主动关节** joint_L1。
+           另外 5 个是 URDF mimic 关节，它们的位置由 robot_state_publisher 从主动
+           关节算出，既不该有 command_interface，也不该进 /joint_states ——
+           声明了反而会出现"同一个自由度被下发两次"。
+           !!! 不声明会怎样（实测）!!!
+           只把夹爪加进 URDF、不加到这里，move_group 会一直刷：
+             The complete state of the robot is not yet known.
+             Missing astribot_gripper_left_joint_L1, astribot_gripper_right_joint_L1
+           **拿不到完整机器人状态 => 规划完全不可用**。也就是说加夹爪这件事一旦
+           只做了模型那一半，现有的所有手臂 demo 会全部停摆，且报错信息指向
+           "状态未知"而不是"你漏配了控制器"，很容易查错方向。 -->
+      <xacro:if value="${use_gripper}">
+        <xacro:astribot_s1_position_joint name="astribot_gripper_left_joint_L1"/>
+        <xacro:astribot_s1_position_joint name="astribot_gripper_right_joint_L1"/>
+      </xacro:if>
     </ros2_control>
     <gazebo>

Commit message: 感知：两台雷达位姿/阈值按实机纠偏，订阅端改 BEST_EFFORT，输入话题参数化
## URDF 雷达安装位姿
原值是 xacro 宏的**占位默认值**，与实机差 0.108 m / 68.8°。已按厂商标定修正，
并做六项几何交叉校验（离地差 2.5mm、两路地面差 0.6mm、间距差 7mm、
高度差一致、连线中点 5.5mm）。

关键认知：驱动通过 SetLivoxLidarInstallAttitude 把外参**写进雷达设备本身**，
所以 /livox/lidar_back 的点已经在 front 系里，上层不要再变换一次。
实测两路 frame_id **都是 livox_frame**（此前文档写「真实 frame 是
livox_mid360_left/right」是错的）。

## SLAM 基准高度：更正我先前的错误答案
camera_init 原点离地 **0.095 m**，不是先前说的 0.017 m。
错因：拿 tf2_echo 读到的 z=0.100 当「实测」，而 TF 只是把 URDF 里的占位值
原样发出来 —— **量一个由错值生成的量，不构成对那个值的验证**。
所以「SLAM 基准不在地面」这个观察是对的。
⬜ 地面平面拟合未做，基准高度只精确到 ±2cm。

## ground_z_min：两台不再同高，共用一个值在数学上不可能同时正确
本节点**不查 TF**，阈值直接作用在雷达自身局部坐标系的原始 z 上，
物理含义 = 「地面在该雷达局部系的 z」+「离地余量」。装得越高就必须越负。
两台安装高度已不同（0.082 vs 0.166），拆成两个值。

## 订阅端 QoS 必须是 BEST_EFFORT
原来写 create_subscription(..., 10)，depth=10 走的是**默认 QoS = RELIABLE**。
仿真里恰好能用（ros_gz_bridge 发 RELIABLE），但实机上游按点云惯例发
BEST_EFFORT，于是 QoS 不兼容、**一帧都收不到**。改用 SensorDataQoS。

## 输入话题名做成参数
hardware_perception.launch.py 原先只覆盖 use_sim_time 就直接 include 仿真那份，
于是实机上订阅了两个**根本不存在**的话题（仿真是 /livox/lidar_{left,right}，
实机是 /livox/lidar_{front,back}）。表现是整条链静默无输出、/scan 一帧都不出，
而每个节点看着都活得好好的。实机现在应传 *_pc2（上一笔的转换节点输出）。

## map→odom（A2 / A3，已实机验证）
· A2 陈旧 TF 检查：**抓到一次真实事件** —— camera_init→aft_mapped 已 1.66s
  未更新（上限 1.00s），正确拒绝发布。此后 78020 次更新无复发。
  机制：tf2 只在某 frame pair 有**新**数据时才修剪缓冲，停更的 pair 会永久
  返回最后一条记录，且 lookup_transform(..., Time()) 一直「成功」、不报错。
· A3 map→camera_init 恒等边改为构造时即发、走 /tf_static（latched）。
  旧代码挂在 _tick 里且只发一次动态 TF，里程计没起时这条边压根不存在，
  晚启动的消费者永远收不到。实证：修复前该边不存在，TF 树是两座孤岛。

新增 test_map_odom_tf_wiring.py(190) 与 test_source_age.py(173)。

Co-Authored-By: Claude <noreply@anthropic.com>

File: ws_robot/src/astribot_s1_description/urdf/astribot_s1.xacro (robot description, xacro)
@@ -26,13 +26,29 @@
        详见 astribot_s1_gripper.xacro 文件头。 -->
   <xacro:arg name="use_gripper" default="true"/>
-  <!-- 双 Livox Mid-360 安装位姿：左前 + 右后对角布局（用户指定），扩大合并视场、
-       减少互相遮挡的盲区（默认值，可外部覆盖）。
-       xyz/rpy 用空格分隔的字符串（xacro origin 惯用写法），改这两个参数即可调整安装位置，
-       不需要碰 astribot_s1_sensors.xacro 里的宏定义本身。
-       坐标约定：torso_base 局部系 +x 朝前、+y 朝左（沿用现有 lidar/camera 挂载点惯例）。 -->
-  <xacro:arg name="livox_left_xyz" default="0.28 0.18 0.10"/>
-  <xacro:arg name="livox_left_rpy" default="0 0 0.4"/>
-  <xacro:arg name="livox_right_xyz" default="-0.28 -0.18 0.10"/>
-  <xacro:arg name="livox_right_rpy" default="0 0 2.74"/>
+  <!-- 双 Livox Mid-360 安装位姿：对角背靠背布局，两台相距约 0.50m、偏航差约 180°，
+       底盘中心恰在两者连线中点。
+       ⚠️ 以下数值是 **2026-09-01 实测/标定推出的**，不是估计值。原来那组
+       （left 0.28 0.18 0.10 / rpy 0 0 0.4，right -0.28 -0.18 0.10 / rpy 0 0 2.74）
+       是 astribot_s1_sensors.xacro 宏的**占位默认值**，与实机差 0.108m / 68.8°。
+       数据来源与交叉校验（三条独立证据一致）：
+       1. 厂商 `/opt/astribot_ros/software/livox_ros_driver2/share/config/MID360_config.json`
+          给出 back(IP .13) 相对 front(IP .12) 的外参：
+          xyz=(1, -496, 84)mm、rpy=(0.0669°, -0.5368°, -178.195°)。
+          注意驱动通过 `SetLivoxLidarInstallAttitude` 把它**写进雷达设备**，
+          所以 `/livox/lidar_back` 发出的点已经在 front 系里了。
+       2. SLAM `mid360.yaml` 的 `chassis_extrinsic_*` 给出 front→chassis：
+          T=(0.17393, 0.16893, 0.082)、R=Rz(-0.800058)。
+       3. 实测地面拟合验证了上面这个 chassis 就是 astribot_torso_base：
+          front 雷达离地实测 0.1745m，由 (1)(2) 推出的预期是 0.1770m，差 2.5mm；
+          两路点云报出的地面高度差 0.0006m；雷达倾角实测 0.43°（外参是纯 Rz，预期 0）。
+          另：两雷达连线中点算出来是 (-0.0036, -0.0042)，即底盘中心确在正中。
+       命名注意：URDF 沿用 left/right，实机话题叫 front/back，对应关系是
+       **left = front = IP 192.168.0.12**，**right = back = IP 192.168.0.13**。
+       改名会牵动自滤配置、gazebo 传感器名与 livox_fusion_node，故本次只改数值。
+       坐标约定：torso_base 局部系 +x 朝前、+y 朝左。 -->
+  <xacro:arg name="livox_left_xyz" default="0.17393 0.16893 0.082"/>
+  <xacro:arg name="livox_left_rpy" default="0 0 -0.800058"/>
+  <xacro:arg name="livox_right_xyz" default="-0.18120 -0.17733 0.166"/>
+  <xacro:arg name="livox_right_rpy" default="0.001168 -0.009370 2.373036"/>
   <!-- controllers_config：ros2_control 控制器 yaml 的绝对路径字符串，
        由调用方（launch.py）用 FindPackageShare + PathJoinSubstitution 拼出后传入，

File: ws_robot/src/astribot_s1_description/urdf/astribot_s1_sensors.xacro (robot description, xacro)
@@ -16,7 +16,11 @@
 <robot xmlns:xacro="http://www.ros.org/wiki/xacro">
   <!-- ================= Livox Mid-360 宏：左右各实例化一次 ================= -->
+  <!-- 宏默认值 = 实机 front(IP .12) 的实测安装位姿。调用方（astribot_s1.xacro）
+       一律显式传 xyz/rpy，所以这里的默认值只在"有人漏传"时兜底 ——
+       原来兜底的是 0.28 0.18 0.10 / 0 0 0.4 那组占位值，与实机差 0.108m/68.8°，
+       漏传时会静默生效，故一并改成实测值。推导与校验见 astribot_s1.xacro 的注释。 -->
   <xacro:macro name="astribot_s1_livox_mid360"
                params="side parent:=astribot_torso_base robot_name:=astribot_s1
-                       xyz:='0.28 0.18 0.10' rpy:='0 0 0.4'">
+                       xyz:='0.17393 0.16893 0.082' rpy:='0 0 -0.800058'">
     <link name="livox_mid360_${side}">
       <inertial>
@@ -44,4 +48,28 @@
       <origin xyz="${xyz}" rpy="${rpy}"/>
     </joint>
+    <!-- ══════════ livox_frame：实机点云真正携带的 frame_id ══════════
+         厂商驱动 launch 里 `frame_id = 'livox_frame'` 是**一个全局值**，
+         于是 /livox/lidar_front 与 /livox/lidar_back 两路点云的 header.frame_id
+         **都是** `livox_frame`（实测，直接解 CDR 取的）。而 TF 树里从来没有
+         这个 frame —— 结果是任何靠 TF 摆放点云的消费者
+         （pointcloud_slice_scan_node 的自滤、livox_fusion_node）在实机上
+         直接查不到变换，而不是"位置略有偏差"。
+         两路共用一个 frame_id 并**不是**厂商的疏漏：驱动通过
+         SetLivoxLidarInstallAttitude 把外参写进雷达设备本身，
+         所以 back 发出的点已经在 front 的坐标系里了（见 MID360_config.json
+         与 livox_extrinsics.yaml 的说明）。也就是说
+             livox_frame ≡ front 雷达坐标系 ≡ livox_mid360_left
+         这条恒等边只是把"实机的命名"接到"URDF 的命名"上。
+         为什么放在 URDF 而不是单独起 static_transform_publisher：
+         RSP 已经在发 /tf_static，多一条边不用多一个进程，也不会出现
+         "同一条边两个源"。只在 side == 左侧那次实例化时发，避免两个父。 -->
+    <xacro:if value="${side == 'left'}">
+      <link name="livox_frame"/>
+      <joint name="livox_frame_joint" type="fixed">
+        <parent link="livox_mid360_${side}"/>
+        <child link="livox_frame"/>
+        <origin xyz="0 0 0" rpy="0 0 0"/>
+      </joint>
+    </xacro:if>
     <gazebo reference="livox_mid360_${side}">
       <sensor name="livox_mid360_${side}_sensor" type="gpu_lidar">
