Commit message: fix(description): preserve camera geometry across capture modes
Record six-camera reference simulation assets and 32 passing model checks. Physical mounts, collision and inertia remain present when capture is disabled. Live navigation and MoveIt camera models agree; all 16 raw camera streams were observed. This records simulation model acceptance, not calibrated hardware or full perception acceptance.

File: ws_robot/src/astribot_s1_description/urdf/astribot_s1.xacro (robot description, xacro)
@@ -15,5 +15,16 @@
   <xacro:arg name="use_lidar" default="true"/>
   <xacro:arg name="use_camera" default="true"/>
-  <xacro:arg name="camera_profile" default="$(find astribot_s1_description)/config/camera_generic.yaml"/>
+  <!-- Navigation only needs the head and torso RGB-D sources.  Wrist/stereo
+       sensors stay opt-in so their render cost cannot starve the two sources
+       that feed the local costmap. -->
+  <xacro:arg name="use_wrist_cameras" default="true"/>
+  <xacro:arg name="use_stereo_cameras" default="true"/>
+  <xacro:arg name="camera_profile" default="$(find astribot_s1_description)/config/camera_head_rgbd.yaml"/>
+  <xacro:arg name="torso_camera_profile" default="$(find astribot_s1_description)/config/camera_torso_rgbd.yaml"/>
+  <xacro:arg name="camera_calibration_dir" default="$(find astribot_s1_description)/config"/>
+  <!-- Empty keeps imported calibration; the warehouse passes a separately
+       versioned provisional layout until physical extrinsics are verified. -->
+  <xacro:arg name="camera_mounts_profile" default=""/>
+  <xacro:arg name="use_native_camera_distortion" default="false"/>
   <!-- use_gripper：是否把平行夹爪作为真实关节模块建模。
        true（默认，与真机一致）：加载 astribot_s1_gripper.xacro，两臂末端各挂
@@ -77,4 +88,7 @@
   <xacro:property name="use_lidar_prop" value="$(arg use_lidar)"/>
   <xacro:property name="use_camera_prop" value="$(arg use_camera)"/>
+  <xacro:property name="use_wrist_cameras_prop" value="$(arg use_wrist_cameras)"/>
+  <xacro:property name="use_stereo_cameras_prop" value="$(arg use_stereo_cameras)"/>
+  <xacro:property name="use_native_camera_distortion_prop" value="$(arg use_native_camera_distortion)"/>
   <xacro:property name="robot_name_prop" value="$(arg robot_name)"/>
   <!-- use_gripper 必须在 include 之前定义成 property：astribot_s1_arm.xacro 在它
@@ -111,7 +125,20 @@
       xyz="$(arg livox_right_xyz)" rpy="$(arg livox_right_rpy)"/>
   </xacro:if>
-  <xacro:if value="${use_camera_prop}">
-    <xacro:astribot_s1_camera parent="astribot_head_link_2" robot_name="${robot_name_prop}" profile="$(arg camera_profile)"/>
-  </xacro:if>
+  <!-- Sensor switches never remove physical camera mass, collision or fixed TF. -->
+  <xacro:property name="camera_capture_enabled" value="${str(use_camera_prop).lower() in ['true', '1']}"/>
+  <xacro:property name="wrist_capture_enabled" value="${camera_capture_enabled and str(use_wrist_cameras_prop).lower() in ['true', '1']}"/>
+  <xacro:property name="stereo_capture_enabled" value="${camera_capture_enabled and str(use_stereo_cameras_prop).lower() in ['true', '1']}"/>
+    <xacro:astribot_s1_calibrated_camera id="head_rgbd" parent="astribot_head_link_2"
+      robot_name="${robot_name_prop}" profile="$(arg camera_profile)" mounts_file="$(arg camera_mounts_profile)" native_distortion="${use_native_camera_distortion_prop}" sensor_enabled="${camera_capture_enabled}"/>
+    <xacro:astribot_s1_calibrated_camera id="torso_rgbd" parent="astribot_torso_base"
+      robot_name="${robot_name_prop}" profile="$(arg torso_camera_profile)" mounts_file="$(arg camera_mounts_profile)" native_distortion="${use_native_camera_distortion_prop}" sensor_enabled="${camera_capture_enabled}"/>
+      <xacro:astribot_s1_calibrated_camera id="left_wrist_rgbd" parent="astribot_arm_left_link_7"
+        robot_name="${robot_name_prop}" profile="$(arg camera_calibration_dir)/camera_left_wrist_rgbd.yaml" mounts_file="$(arg camera_mounts_profile)" native_distortion="${use_native_camera_distortion_prop}" sensor_enabled="${wrist_capture_enabled}"/>
+      <xacro:astribot_s1_calibrated_camera id="right_wrist_rgbd" parent="astribot_arm_right_link_7"
+        robot_name="${robot_name_prop}" profile="$(arg camera_calibration_dir)/camera_right_wrist_rgbd.yaml" mounts_file="$(arg camera_mounts_profile)" native_distortion="${use_native_camera_distortion_prop}" sensor_enabled="${wrist_capture_enabled}"/>
+      <xacro:astribot_s1_calibrated_camera id="head_stereo_left" parent="astribot_head_link_2"
+        robot_name="${robot_name_prop}" profile="$(arg camera_calibration_dir)/camera_head_stereo_left.yaml" mounts_file="$(arg camera_mounts_profile)" native_distortion="${use_native_camera_distortion_prop}" sensor_enabled="${stereo_capture_enabled}"/>
+      <xacro:astribot_s1_calibrated_camera id="head_stereo_right" parent="head_stereo_left_camera_optical_frame"
+        robot_name="${robot_name_prop}" profile="$(arg camera_calibration_dir)/camera_head_stereo_right.yaml" mounts_file="$(arg camera_mounts_profile)" native_distortion="${use_native_camera_distortion_prop}" sensor_enabled="${stereo_capture_enabled}"/>
   <!-- ============ ros2_control + gz_ros2_control 插件 ============ -->
   <!-- wheel_effort_limit 不再传进 astribot_s1_ros2_control 宏——实测发现

File: ws_robot/src/astribot_s1_description/urdf/astribot_s1_sensors.xacro (robot description, xacro)
@@ -123,4 +123,67 @@
     </gazebo>
   </xacro:macro>
+  <!-- Calibrated camera instance.  Names are prefixed by id so all six
+       firmware cameras can coexist in one model without frame/sensor clashes. -->
+  <xacro:macro name="astribot_s1_calibrated_camera" params="id parent robot_name profile native_distortion:=false mounts_file:='' sensor_enabled:=true">
+    <xacro:property name="camera" value="${xacro.load_yaml(profile)}"/>
+    <xacro:property name="mount" value="${xacro.load_yaml(mounts_file)['cameras'][id] if mounts_file else camera}"/>
+    <xacro:property name="housing_size" value="${mount.get('housing_size', '0.03 0.08 0.03')}"/>
+    <!-- camera_link is the entrance pupil. Housing belongs behind that plane,
+         not around the sensor origin, otherwise it can occlude its own lens. -->
+    <xacro:property name="housing_center" value="${mount.get('housing_center_xyz', '-0.016 0 0')}"/>
+    <link name="${id}_camera_link">
+      <inertial><origin xyz="${housing_center}"/><mass value="0.05"/><inertia ixx="0.00001" ixy="0" ixz="0" iyy="0.00001" iyz="0" izz="0.00001"/></inertial>
+      <visual><origin xyz="${housing_center}"/><geometry><box size="${housing_size}"/></geometry><material name="astribot_camera_color"><color rgba="0.05 0.05 0.05 1"/></material></visual>
+      <!-- An override may omit only volume already represented by the fixed
+           parent's collision geometry; the reference profile tests this union. -->
+      <collision><origin xyz="${mount.get('collision_housing_center_xyz', housing_center)}"/><geometry><box size="${mount.get('collision_housing_size', housing_size)}"/></geometry></collision>
+      <xacro:if value="${'mount_bracket_size' in mount}">
+        <visual name="${id}_mount_bracket">
+          <origin xyz="${mount.mount_bracket_center_xyz}"/>
+          <geometry><box size="${mount.mount_bracket_size}"/></geometry>
+          <material name="astribot_camera_bracket_color"><color rgba="0.45 0.45 0.45 1"/></material>
+        </visual>
+        <xacro:if value="${mount.get('mount_bracket_collision', True)}">
+          <collision name="${id}_mount_bracket_collision">
+            <origin xyz="${mount.mount_bracket_center_xyz}"/>
+            <geometry><box size="${mount.mount_bracket_size}"/></geometry>
+          </collision>
+        </xacro:if>
+      </xacro:if>
+    </link>
+    <joint name="${id}_camera_joint" type="fixed">
+      <parent link="${mount.get('parent_frame', parent)}"/><child link="${id}_camera_link"/>
+      <origin xyz="${mount.mount_xyz}" rpy="${mount.mount_rpy}"/>
+    </joint>
+    <link name="${id}_camera_optical_frame"/>
+    <joint name="${id}_camera_optical_joint" type="fixed">
+      <parent link="${id}_camera_link"/><child link="${id}_camera_optical_frame"/>
+      <origin xyz="0 0 0" rpy="-1.5707963267948966 0 -1.5707963267948966"/>
+    </joint>
+    <!-- Installed housing and fixed frames remain present when capture is disabled. -->
+    <xacro:if value="${sensor_enabled}">
+    <gazebo reference="${id}_camera_link">
+      <sensor name="${id}_sensor" type="${camera.sensor_type}">
+        <pose>0 0 0 0 0 0</pose>
+        <topic>${'/model/' + robot_name + '/' + id if camera.sensor_type == 'rgbd_camera' else '/model/' + robot_name + '/' + id + '/image_raw'}</topic>
+        <update_rate>${camera.rate_hz}</update_rate><always_on>true</always_on><visualize>false</visualize>
+        <camera>
+          <horizontal_fov>${camera.horizontal_fov}</horizontal_fov>
+          <image><width>${camera.width}</width><height>${camera.height}</height><format>R8G8B8</format></image>
+          <clip><near>${camera.near_m}</near><far>${camera.far_m}</far></clip>
+          <xacro:if value="${native_distortion}">
+            <!-- YAML follows ROS/OpenCV order k1,k2,p1,p2,k3; SDF uses k1,k2,k3,p1,p2. -->
+            <distortion>
+              <k1>${camera.distortion[0]}</k1><k2>${camera.distortion[1]}</k2><k3>${camera.distortion[4]}</k3>
+              <p1>${camera.distortion[2]}</p1><p2>${camera.distortion[3]}</p2>
+              <center>${camera.intrinsics.color[2] / camera.width} ${camera.intrinsics.color[5] / camera.height}</center>
+            </distortion>
+          </xacro:if>
+        </camera>
+      </sensor>
+    </gazebo>
+    </xacro:if>
+  </xacro:macro>
+  <!-- Legacy single head camera entry point retained for downstream launch files. -->
   <xacro:macro name="astribot_s1_camera" params="parent:=astribot_head_link_2 robot_name:=astribot_s1 profile">
     <xacro:property name="camera" value="${xacro.load_yaml(profile)}"/>

Commit message: Add explicit READY initialization for navigation simulation
Keep the default posture unchanged and validate the exact position-command joints before starting Gazebo. Archive 16 offline checks and measured 22-joint initialization evidence. The first-stage task remains unaccepted after MTC_SCENE_CHANGED; zero-to-READY motion is a separate paused issue.

File: ws_robot/src/astribot_s1_description/urdf/astribot_s1.xacro (robot description, xacro)
@@ -67,4 +67,7 @@
        本文件内部不出现任何硬编码路径。 -->
   <xacro:arg name="controllers_config" default=""/>
+  <xacro:arg name="sim_initial_positions_file" default=""/>
+  <xacro:property name="sim_initial_positions_file" value="$(arg sim_initial_positions_file)"/>
+  <xacro:property name="sim_initial_positions" value="${xacro.load_yaml(sim_initial_positions_file)['initial_positions'] if sim_initial_positions_file else dict()}"/>
   <!-- 全向轮力矩闭环驱动改造新增：轮子effort硬件接口边界 + 几何半径统一从这里
        外部传入，禁止在 torso_wheel/ros2_control xacro 里写死。

File: ws_robot/src/astribot_s1_description/urdf/astribot_s1_ros2_control.xacro (robot description, xacro)
@@ -22,5 +22,9 @@
     <joint name="${name}">
       <command_interface name="position"/>
-      <state_interface name="position"/>
+      <state_interface name="position">
+        <xacro:if value="${name in sim_initial_positions}">
+          <param name="initial_value">${sim_initial_positions[name]}</param>
+        </xacro:if>
+      </state_interface>
       <state_interface name="velocity"/>
       <state_interface name="effort"/>
