Commit message: Fix real-run issues found while actually launching the simulation
联调实测发现并修复的问题（均为运行时实测暴露，非纸面审查）：
- aws_robomaker_warehouse_GroundB_01/RoofB_01 官方 model.sdf 惯性张量违反三角不等式，
  新版 Ignition Gazebo(Fortress) 直接拒绝加载世界；不修改 submodule，
  改为在 astribot_s1_gazebo_bringup/models/ 下放置资源路径优先级更高的覆盖版 model.sdf
  （只改惯性张量，mesh/材质仍引用 submodule 原始文件）
- robot_description 参数需要 ParameterValue(..., value_type=str) 包装，否则被当 YAML 解析报错
- MecanumDrive 的 <topic> 是字面量话题名，不像 OdometryPublisher 会自动加 /model/<name>/ 前缀，
  显式改成绝对话题名与 ros_gz_bridge 对齐；OdometryPublisher 则改回默认行为
  （之前误加 <odom_topic>/<tf_topic> 反而导致它完全不发布）
- 5个ros2_control控制器spawner并行拉起会偶发 controller_manager 服务并发竞争导致加载失败，
  改成单个 spawner 进程串行加载全部控制器
- 新增 ROS_DOMAIN_ID 隔离（默认42），避免和同一台机器上任何其它无关 ROS2 图撞话题/服务名
  （实测复现过：另一个无关工作空间的 robot_state_publisher 用 transient_local QoS
  抢答了 /robot_description 订阅）
- GZ_SIM_RESOURCE_PATH 补充 astribot_s1_description 包 share 目录的父路径，
  修复机器人自身 mesh 在 Gazebo GUI 里 package://->model:// 转换后加载失败的问题

已知残留问题（未解决，见对话说明）：麦克纳姆轮在收到 /cmd_vel 后确认会旋转
（已用 ign model -l 验证轮子姿态角持续变化），但底盘整体不产生平移——
根因判断是简化圆柱碰撞体(各向同性摩擦 mu1=mu2=1.0)无法复现真实麦克纳姆轮
滚子结构的各向异性摩擦效果，需要后续用 <fdir1>+差异化 mu1/mu2 调整摩擦各向异性。

Co-Authored-By: Claude <noreply@anthropic.com>

File: ws_robot/src/astribot_s1_description/urdf/astribot_s1.gazebo.xacro (robot description, xacro)
@@ -12,9 +12,15 @@
 -->
 <robot xmlns:xacro="http://www.ros.org/wiki/xacro">
-  <xacro:macro name="astribot_s1_gazebo_chassis_plugins" params="wheel_radius:=0.08 wheel_separation:=0.4327 wheelbase:=0.4327">
+  <xacro:macro name="astribot_s1_gazebo_chassis_plugins"
+               params="robot_name:=astribot_s1 wheel_radius:=0.08 wheel_separation:=0.4327 wheelbase:=0.4327">
     <!-- ========== 麦克纳姆全向轮驱动：官方 MecanumDrive 系统插件，天然支持 x/y/yaw 三自由度 ==========
          与 astribot_chassis.yaml 里 astribot_chassis_x/y/z_rot 三个独立自由度的抽象完全对应。
          订阅话题 /model/<robot_name>/cmd_vel(geometry_msgs/Twist，含 linear.y 侧移分量)，
-         发布 /model/<robot_name>/odometry(gz.msgs.Odometry)——由 ros_gz_bridge 转成 ROS2 话题。 -->
+         发布 /model/<robot_name>/odometry(gz.msgs.Odometry)——由 ros_gz_bridge 转成 ROS2 话题。
+         !!! 实测踩坑记录 !!!：MecanumDrive 的 <topic> 只要显式写了，就是"字面量"话题名，
+         不会像 OdometryPublisher 的 <odom_topic> 那样自动补上 "/model/<name>/" 前缀
+         （本方案联调时验证过：不写绝对路径会导致 /cmd_vel 消息桥接过去后机器人纹丝不动，
+         因为插件实际订阅的是裸的 "cmd_vel"，跟 ros_gz_bridge 转发目标 "/model/<name>/cmd_vel"
+         对不上）。所以这里显式写成和 ros_gz_bridge 配置一致的绝对话题名。 -->
     <gazebo>
       <plugin filename="gz-sim-mecanum-drive-system" name="gz::sim::systems::MecanumDrive">
@@ -38,10 +44,16 @@
         <min_jerk>-50.0</min_jerk>
         <max_jerk>50.0</max_jerk>
-        <topic>cmd_vel</topic>
-        <odom_topic>odometry</odom_topic>
+        <topic>/model/${robot_name}/cmd_vel</topic>
+        <odom_topic>/model/${robot_name}/odometry</odom_topic>
         <frame_id>odom</frame_id>
         <child_frame_id>astribot_torso_base</child_frame_id>
       </plugin>
-      <!-- MecanumDrive 本身不发布 TF（已知限制），单独挂 OdometryPublisher 补 /tf 与 nav_msgs/Odometry -->
+      <!-- MecanumDrive 本身不发布 TF（已知限制），单独挂 OdometryPublisher 补 /tf 与 nav_msgs/Odometry。
+           !!! 实测踩坑记录 !!!：一开始仿照 MecanumDrive 那样给它加了显式的
+           <odom_topic>/<tf_topic> 绝对路径，结果这个插件直接不再发布任何东西了
+           （<odom_topic>不是 OdometryPublisher 认识的标签名，多出来的未知子标签让这个
+           plugin 加载/解析出了问题）。OdometryPublisher 自己的默认行为就是按
+           "/model/<模型名>/odometry"、"/model/<模型名>/tf" 这样自动加前缀发布
+           （已实测验证过默认行为正确），所以这里保持默认，不要再加那两个标签。 -->
       <plugin filename="gz-sim-odometry-publisher-system" name="gz::sim::systems::OdometryPublisher">
         <!-- 兼容提示：ignition-gazebo-odometry-publisher-system /

File: ws_robot/src/astribot_s1_description/urdf/astribot_s1.xacro (robot description, xacro)
@@ -39,4 +39,5 @@
   <xacro:astribot_s1_ros2_control controllers_config="$(arg controllers_config)"/>
   <!-- ============ 底盘全向轮驱动 + 里程计 + 轮子摩擦 ============ -->
-  <xacro:astribot_s1_gazebo_chassis_plugins wheel_radius="0.08" wheel_separation="0.4327" wheelbase="0.4327"/>
+  <xacro:astribot_s1_gazebo_chassis_plugins
+    robot_name="${robot_name_prop}" wheel_radius="0.08" wheel_separation="0.4327" wheelbase="0.4327"/>
 </robot>

Commit message: Add dual Livox Mid-360 lidars + SLAM Toolbox mapping/localization stack
新增/改动内容：
- astribot_s1_description: 原单个通用2D雷达替换为两个 Livox Mid-360
  (livox_mid360_left 左前 / livox_mid360_right 右后对角安装，用户指定位置，
  xacro参数化可调)，用 gpu_lidar 近似真实360°x59°FOV仿真，明确标注这是近似
  而非真实非重复扫描花纹(gz-sim无官方Mid-360仿真插件)。
- astribot_s1_gazebo_bringup: 双雷达PointCloud2桥接；新增
  gz-sim-sensors-system插件修复(联调中发现aws world无任何plugin标签，
  导致所有camera/gpu_lidar包括头部相机此前一直发布不出数据)；新增
  static_transform_publisher给3个传感器做frame_id别名(gz-sim传感器消息
  frame_id是model/link/sensor长路径，TF树里没有这个frame)。
- 新增 astribot_s1_perception 包(ament_python)：
  - livox_preprocess_node/livox_fusion_node: 直通/半径/地面滤波 + 时间同步
    + tf2坐标变换融合，如实标注仿真侧无逐点时间戳、不做完整逐点去畸变
  - 6个launch文件区分仿真/硬件分支、mapping/localization两种SLAM模式，
    顶层 perception_slam_bringup.launch.py 用 env/mode 参数切换四种组合
  - SLAM Toolbox建图/定位参数、pointcloud_to_laserscan投影参数、
    双雷达外参文档、真实driver的MID360 JSON配置(IP占位)
- livox_ros_driver2 以 git submodule 接入(硬件分支)，用户提供sudo密码后
  实际完成 Livox-SDK2 源码编译安装 + livox_ros_driver2 colcon build 通过
  (而不是原计划的COLCON_IGNORE兜底方案)，自带 prepare_livox_driver2.sh
  安全准备脚本(不用官方build.sh，那个会rm -rf整个工作空间build/install)。

仿真分支已实测走通建图+定位两种模式全链路（/livox/lidar_left|right →
预处理 → 融合 → /scan → SLAM Toolbox → /map，serialize_map保存后
localization模式重新加载验证），联调中额外发现并修复3个真实bug，
详见 astribot_s1_perception/README_PERCEPTION.md 第7节。

Co-Authored-By: Claude <noreply@anthropic.com>

File: ws_robot/src/astribot_s1_description/urdf/astribot_s1.gazebo.xacro (robot description, xacro)
@@ -64,4 +64,20 @@
         <dimensions>3</dimensions>
       </plugin>
+      <!-- !!! 实测踩坑记录（新增，非常关键）!!!：aws_robomaker_small_warehouse_world 的
+           world 文件本身一个 <plugin> 标签都没有，gz-sim 找不到 world 级插件配置时，
+           会退回 ~/.gz(或.ignition)/sim/<ver>/server.config 里的默认系统插件列表——
+           实测那份默认列表只有 Physics/UserCommands/SceneBroadcaster 三个，
+           **没有 Sensors 系统**！缺了它，机器人身上所有 camera/gpu_lidar 传感器
+           （包括这里新加的双 Livox Mid-360，也包括头部相机）只会被解析、
+           永远不会真正渲染/发布任何数据——话题能在 `ros2 topic list` 里看到，
+           但 `ros2 topic hz` 永远拿不到消息，很容易被误判成"话题名/桥接配置错了"。
+           因为不允许修改 aws 官方仓库的 world 文件，这里改成把 Sensors 系统插件挂在
+           "我们自己机器人模型"的 <gazebo> 标签下——gz-sim 的 Sensors 系统一旦在
+           场景里任意实体上加载成功，就会全局接管整个仿真里所有传感器的渲染，
+           不需要非挂在 world 实体上不可，这是应对"不能改 world 文件"场景的标准做法。 -->
+      <plugin filename="gz-sim-sensors-system" name="gz::sim::systems::Sensors">
+        <!-- 兼容提示：ignition-gazebo-sensors-system / ignition::gazebo::systems::Sensors -->
+        <render_engine>ogre2</render_engine>
+      </plugin>
     </gazebo>
     <!-- 四个轮子摩擦系数：提高地面附着力，避免全向轮"打滑不走直线" -->

File: ws_robot/src/astribot_s1_description/urdf/astribot_s1.xacro (robot description, xacro)
@@ -3,5 +3,5 @@
   文件用途：Astribot S1 轮式双臂机器人 —— 顶层 xacro 入口。
   聚合：底盘(4麦克纳姆轮+4自由度升降躯干) + 头部(2自由度) + 左右机械臂(各7自由度)
-       + 可选传感器(2D激光雷达/RGB相机) + ros2_control + Gazebo 插件。
+       + 可选传感器(双 Livox Mid-360 3D激光雷达/RGB相机) + ros2_control + Gazebo 插件。
   用法（供 launch.py 调用，见 astribot_s1_gazebo_bringup/launch/warehouse_sim.launch.py）：
     xacro astribot_s1.xacro robot_name:=astribot_s1 use_lidar:=true use_camera:=true \
@@ -15,4 +15,13 @@
   <xacro:arg name="use_lidar" default="true"/>
   <xacro:arg name="use_camera" default="true"/>
+  <!-- 双 Livox Mid-360 安装位姿：左前 + 右后对角布局（用户指定），扩大合并视场、
+       减少互相遮挡的盲区（默认值，可外部覆盖）。
+       xyz/rpy 用空格分隔的字符串（xacro origin 惯用写法），改这两个参数即可调整安装位置，
+       不需要碰 astribot_s1_sensors.xacro 里的宏定义本身。
+       坐标约定：torso_base 局部系 +x 朝前、+y 朝左（沿用现有 lidar/camera 挂载点惯例）。 -->
+  <xacro:arg name="livox_left_xyz" default="0.28 0.18 0.10"/>
+  <xacro:arg name="livox_left_rpy" default="0 0 0.4"/>
+  <xacro:arg name="livox_right_xyz" default="-0.28 -0.18 0.10"/>
+  <xacro:arg name="livox_right_rpy" default="0 0 2.74"/>
   <!-- controllers_config：ros2_control 控制器 yaml 的绝对路径字符串，
        由调用方（launch.py）用 FindPackageShare + PathJoinSubstitution 拼出后传入，
@@ -30,6 +39,13 @@
   <xacro:include filename="$(find astribot_s1_description)/urdf/astribot_s1.gazebo.xacro"/>
   <!-- ============ 传感器（按参数开关，默认都打开） ============ -->
+  <!-- 双 Livox Mid-360：分别实例化 left/right，frame_id 各自独立
+       （livox_mid360_left / livox_mid360_right，不共用同一个 frame_id）。 -->
   <xacro:if value="${use_lidar_prop}">
-    <xacro:astribot_s1_lidar parent="astribot_torso_base" robot_name="${robot_name_prop}"/>
+    <xacro:astribot_s1_livox_mid360
+      side="left" parent="astribot_torso_base" robot_name="${robot_name_prop}"
+      xyz="$(arg livox_left_xyz)" rpy="$(arg livox_left_rpy)"/>
+    <xacro:astribot_s1_livox_mid360
+      side="right" parent="astribot_torso_base" robot_name="${robot_name_prop}"
+      xyz="$(arg livox_right_xyz)" rpy="$(arg livox_right_rpy)"/>
   </xacro:if>
   <xacro:if value="${use_camera_prop}">

File: ws_robot/src/astribot_s1_description/urdf/astribot_s1_sensors.xacro (robot description, xacro)
@@ -1,19 +1,31 @@
 <?xml version="1.0"?>
 <!--
-  文件用途：可选传感器（2D 激光雷达 + RGB 相机），用 xacro:if 通过顶层参数 use_lidar/use_camera 开关。
-  雷达装在底盘前方（astribot_torso_base 前沿），相机装在头部 astribot_head_link_2（随头部俯仰转动）。
-  均使用 Gazebo 官方 gz-sim 传感器插件（非实验性），通过 ros_gz_bridge 转出标准 ROS2 话题
-  （見 astribot_s1_gazebo_bringup/config/astribot_s1_bridge.yaml）。
+  文件用途：机器人自身携带的传感器 —— 双 Livox Mid-360 3D 激光雷达 + 头部 RGB 相机。
+  用 xacro:if 通过顶层参数 use_lidar/use_camera 开关。均使用 Gazebo 官方 gz-sim 传感器插件
+  （非实验性），通过 ros_gz_bridge 转出标准 ROS2 话题（見
+  astribot_s1_gazebo_bringup/launch/warehouse_sim.launch.py 里的 bridge_args）。
+  ============================ Livox Mid-360 仿真说明（务必先读） ============================
+  实测确认：Ignition/Gz Sim 目前没有官方或主流维护的 Mid-360 真实"非重复花瓣扫描"仿真插件
+  （官方 livox_laser_simulation 仓库只支持 Gazebo Classic，没有 gz-sim 移植版）。
+  本方案采用社区通用做法：用 gz-sim 原生 <sensor type="gpu_lidar"> 配置成与 Mid-360 规格
+  一致的视场角（水平360°、垂直 -7°~+52°共59°）来近似，输出标准 PointCloud2 点云，
+  在数据链路和下游算法层面与真实 Mid-360 等价，但不是逐点还原真实花瓣扫描图案——
+  这一点在 astribot_s1_perception 包的 README 里也会再次说明，避免误认为是精确仿真。
+  ============================================================================================
 -->
 <robot xmlns:xacro="http://www.ros.org/wiki/xacro">
-  <xacro:macro name="astribot_s1_lidar" params="parent:=astribot_torso_base robot_name:=astribot_s1">
-    <link name="lidar_link">
+  <!-- ================= Livox Mid-360 宏：左右各实例化一次 ================= -->
+  <xacro:macro name="astribot_s1_livox_mid360"
+               params="side parent:=astribot_torso_base robot_name:=astribot_s1
+                       xyz:='0.28 0.18 0.10' rpy:='0 0 0.4'">
+    <link name="livox_mid360_${side}">
       <inertial>
-        <mass value="0.15"/>
-        <inertia ixx="0.0001" ixy="0" ixz="0" iyy="0.0001" iyz="0" izz="0.0001"/>
+        <!-- 官方规格：65x65x60mm, 265g -->
+        <mass value="0.265"/>
+        <inertia ixx="0.00015" ixy="0" ixz="0" iyy="0.00015" iyz="0" izz="0.00012"/>
       </inertial>
       <visual>
         <geometry>
-          <cylinder radius="0.035" length="0.04"/>
+          <cylinder radius="0.0325" length="0.06"/>
         </geometry>
         <material name="astribot_lidar_color">
@@ -23,20 +35,20 @@
       <collision>
         <geometry>
-          <cylinder radius="0.035" length="0.04"/>
+          <cylinder radius="0.0325" length="0.06"/>
         </geometry>
       </collision>
     </link>
-    <!-- 装在底盘前沿（+x 方向）、略高于地面，避免与底盘外壳碰撞体自相交 -->
-    <joint name="lidar_joint" type="fixed">
+    <joint name="livox_mid360_${side}_joint" type="fixed">
       <parent link="${parent}"/>
-      <child link="lidar_link"/>
-      <origin xyz="0.30 0 0.05" rpy="0 0 0"/>
+      <child link="livox_mid360_${side}"/>
+      <origin xyz="${xyz}" rpy="${rpy}"/>
     </joint>
-    <gazebo reference="lidar_link">
-      <sensor name="astribot_lidar" type="gpu_lidar">
+    <gazebo reference="livox_mid360_${side}">
+      <sensor name="livox_mid360_${side}_sensor" type="gpu_lidar">
         <pose>0 0 0 0 0 0</pose>
-        <!-- 用带 robot_name 的绝对话题名(以 / 开头)，避免 gz-sim 按 world/model/link/sensor
-             层级自动生成一长串话题名——绝对名字才能在 bridge yaml 里写死映射关系 -->
-        <topic>/model/${robot_name}/scan</topic>
+        <!-- 绝对话题名，gz-sim 会在其后缀 "/points" 输出 gz.msgs.PointCloudPacked 点云
+             （对应 ros_gz_bridge 里 .../points@sensor_msgs/msg/PointCloud2[gz.msgs.PointCloudPacked
+             的桥接写法，见 warehouse_sim.launch.py）。 -->
+        <topic>/model/${robot_name}/livox_mid360_${side}</topic>
         <update_rate>10</update_rate>
         <always_on>true</always_on>
@@ -45,13 +57,24 @@
           <scan>
             <horizontal>
-              <samples>360</samples>
+              <!-- 水平 360°，采样数按 Mid-360 单帧约 20000 点(10Hz下等效200000pts/s)量级近似取，
+                   实测如果卡顿可调低（见 astribot_s1_perception/README_PERCEPTION.md 里的降采样建议）。 -->
+              <samples>400</samples>
               <resolution>1</resolution>
               <min_angle>-3.14159</min_angle>
               <max_angle>3.14159</max_angle>
             </horizontal>
+            <vertical>
+              <!-- Mid-360 真实垂直视场 -7°~+52°(共59°)，换算弧度：-0.1222 ~ 0.9076 -->
+              <samples>32</samples>
+              <resolution>1</resolution>
+              <min_angle>-0.1222</min_angle>
+              <max_angle>0.9076</max_angle>
+            </vertical>
           </scan>
           <range>
-            <min>0.12</min>
-            <max>12.0</max>
+            <!-- 官方规格：盲区0.1~0.2m，最远70m(高反射率)；仿真里取中间值，太远会引入仓储世界
+                 外墙/屋顶的无效远点，拖慢下游点云处理 -->
+            <min>0.10</min>
+            <max>40.0</max>
             <resolution>0.01</resolution>
           </range>

Commit message: 修复麦克纳姆轮平移bug + 新增自主巡游建图节点
底盘曾存在两个真实bug：轮子转身体不平移、平移过程中身体会缓慢倾倒。
排查确认为4个独立根因（均实测复现+验证，非纸面推演）：

1. 各向异性摩擦近似在0.08m小尺寸轮子上失效（已有记录，本次未改）。
2. VelocityControl直接设定车身速度，MecanumDrive仍按真实摩擦假设独立算
   轮速，两者速度不一致的部分通过轮地摩擦力反馈到车身没人管的z/roll/pitch
   自由度，几十秒到一两分钟内缓慢累积成倾斜姿态。修复：四个轮子mu1/mu2
   清零，完全解耦两个插件。
3. 双Mid-360打在机器人自己身上的固定结构(0.10~0.25m)被巡游节点误判成
   "到处都是障碍物"，一直原地自转走不出去。修复：pointcloud_filter_params
   的range_min从0.15提到0.35。
4. autonomous_patrol_node把车体系角度直接当world系角度发cmd_vel，但
   VelocityControl插件二进制内部组件类型是WorldLinearVelocityCmdTag，
   按world系解释——车身同时自转导致推力方向连续扫过整圈、互相抵消。
   修复：新增/odom订阅换算当前航向角，body角度+yaw再算vx/vy。

新增 autonomous_patrol_node：反应式漫游（找最开阔方向平移+缓慢自转扩大
覆盖），带跟随移动方向的碰撞安全扇区、全向最近距离紧急阈值、基于/odom的
姿态异常安全监控（作为对上述根因修复的工程纵深防御，非替代）。

最终验证：单实例连续运行22+分钟，z稳定在0.1342m标称值，roll/pitch全程0，
安全监控零触发，/map栅格从274x232增长到274x282。

Co-Authored-By: Claude <noreply@anthropic.com>

File: ws_robot/src/astribot_s1_description/urdf/astribot_s1.gazebo.xacro (robot description, xacro)
@@ -14,14 +14,31 @@
   <xacro:macro name="astribot_s1_gazebo_chassis_plugins"
                params="robot_name:=astribot_s1 wheel_radius:=0.08 wheel_separation:=0.4327 wheelbase:=0.4327">
-    <!-- ========== 麦克纳姆全向轮驱动：官方 MecanumDrive 系统插件，天然支持 x/y/yaw 三自由度 ==========
-         与 astribot_chassis.yaml 里 astribot_chassis_x/y/z_rot 三个独立自由度的抽象完全对应。
-         订阅话题 /model/<robot_name>/cmd_vel(geometry_msgs/Twist，含 linear.y 侧移分量)，
-         发布 /model/<robot_name>/odometry(gz.msgs.Odometry)——由 ros_gz_bridge 转成 ROS2 话题。
-         !!! 实测踩坑记录 !!!：MecanumDrive 的 <topic> 只要显式写了，就是"字面量"话题名，
-         不会像 OdometryPublisher 的 <odom_topic> 那样自动补上 "/model/<name>/" 前缀
-         （本方案联调时验证过：不写绝对路径会导致 /cmd_vel 消息桥接过去后机器人纹丝不动，
-         因为插件实际订阅的是裸的 "cmd_vel"，跟 ros_gz_bridge 转发目标 "/model/<name>/cmd_vel"
-         对不上）。所以这里显式写成和 ros_gz_bridge 配置一致的绝对话题名。 -->
+    <!-- ========== 底盘全向驱动：VelocityControl(实际驱动身体位移) + MecanumDrive(轮子视觉旋转) ==========
+         !!! 实测踩坑记录（麦克纳姆轮"轮子转、车不走"bug 的完整排查过程）!!!
+         第一轮尝试：给四个轮子配置各向异性摩擦（fdir1 按 45°对角线 + mu2=0，完全照抄
+         gz-sim 官方示例 `/usr/share/ignition/ignition-gazebo6/worlds/mecanum_drive.sdf`
+         的写法，连碰撞体形状都改成官方示例用的球体）。结果实测：
+           - 直接跑官方示例：车辆确实产生了平移（验证这套摩擦方案在本机物理引擎下可行）；
+           - 把官方示例的轮子等比例缩小到接近我们机器人的尺寸(半径0.3m→0.075m)后
+             重新测试同一份官方示例：**平移消失了**——证明这不是我们的配置错误，
+             而是 gz-sim6(Fortress)+DART 物理引擎组合下，这套"各向异性摩擦"近似方案本身
+             在小尺寸轮子上会失效（大概率是接触点计算/摩擦锥在小尺寸下数值不稳定，
+             不是文档记录的已知限制，是本方案实测发现的）。本机器人轮子半径只有0.08m，
+             正好落在这个失效区间内，所以无论怎么调摩擦系数/坐标系表达都不会有效果。
+         第二轮修复（本方案最终采用）：改用 gz-sim 官方 `VelocityControl` 系统插件
+         （示例：`/usr/share/ignition/ignition-gazebo6/worlds/velocity_control.sdf`）
+         ——它不依赖轮子-地面摩擦力学，而是直接对模型本体设置线速度/角速度，
+         从根本上绕开了"小尺寸轮子摩擦近似失效"这个物理引擎数值问题，实测在本机器人
+         真实质量(39kg躯干)和真实轮子尺寸(0.08m)下 x/y/yaw 三个自由度平移旋转都正常。
+         MecanumDrive 插件保留下来，只用来让轮子按论理转速转起来做视觉效果
+         （它自己单独驱动的车身位移量在我们的尺寸下可忽略不计，不会和 VelocityControl
+         的真实位移打架，两者互不干扰，同时生效）。 -->
     <gazebo>
+      <plugin filename="gz-sim-velocity-control-system" name="gz::sim::systems::VelocityControl">
+        <!-- 兼容提示：ignition-gazebo-velocity-control-system /
+             ignition::gazebo::systems::VelocityControl。
+             没有 <topic> 子标签可配置——它固定订阅 "/model/<模型名>/cmd_vel"
+             （官方示例验证过，和 ros_gz_bridge 里桥接的目标话题名天然一致，不用额外配置）。 -->
+      </plugin>
       <plugin filename="gz-sim-mecanum-drive-system" name="gz::sim::systems::MecanumDrive">
         <!-- 兼容提示（旧版 Ignition Gazebo Fortress 早期/自编译环境可能仍需要这两行写法）：
@@ -44,10 +61,15 @@
         <min_jerk>-50.0</min_jerk>
         <max_jerk>50.0</max_jerk>
+        <!-- !!! 实测踩坑记录 !!!：MecanumDrive 的 <topic> 只要显式写了，就是"字面量"话题名，
+             不会像 OdometryPublisher 的 <odom_topic> 那样自动补上 "/model/<name>/" 前缀，
+             必须显式写成和 ros_gz_bridge 配置一致的绝对话题名，否则订阅不到消息。 -->
         <topic>/model/${robot_name}/cmd_vel</topic>
-        <odom_topic>/model/${robot_name}/odometry</odom_topic>
+        <odom_topic>/model/${robot_name}/mecanum_odometry</odom_topic>
         <frame_id>odom</frame_id>
         <child_frame_id>astribot_torso_base</child_frame_id>
       </plugin>
-      <!-- MecanumDrive 本身不发布 TF（已知限制），单独挂 OdometryPublisher 补 /tf 与 nav_msgs/Odometry。
+      <!-- MecanumDrive/VelocityControl 都不发布可靠的 TF，单独挂 OdometryPublisher 补
+           /tf 与 nav_msgs/Odometry（它是基于模型真实位姿变化算出来的，不受上面选用哪个
+           驱动插件影响）。
            !!! 实测踩坑记录 !!!：一开始仿照 MecanumDrive 那样给它加了显式的
            <odom_topic>/<tf_topic> 绝对路径，结果这个插件直接不再发布任何东西了
@@ -81,20 +103,38 @@
       </plugin>
     </gazebo>
-    <!-- 四个轮子摩擦系数：提高地面附着力，避免全向轮"打滑不走直线" -->
+    <!-- !!! 实测踩坑记录（第三轮，真正的"平移正常但会慢慢倾倒"根因）!!!：上一版本把
+         四个轮子摩擦系数恢复成普通各向同性摩擦(mu1=mu2=1.0)，理由是"轮子不再负责实际
+         驱动身体位移，只是给轮子一个合理的地面摩擦力，避免打滑的观感问题"——这个理由
+         本身是错的。MecanumDrive 插件仍然在**独立**按照它自己内部的全向轮运动学公式
+         计算并驱动四个轮子关节的转速（只是为了让轮子在视觉上转得"看起来对"），这个转速
+         是按"轮子和地面之间存在真实摩擦、靠摩擦力驱动车身"这个假设算出来的；但车身实际
+         的位移是由 VelocityControl 直接设定的，和轮子转速隐含的"应有位移"并不是同一回事
+         （两者独立计算，几乎不可能完全一致）。只要轮子还有摩擦(mu1/mu2>0)，这个"轮子
+         转速暗示的运动"和"车身实际被强制的运动"之间的差异，就会在每一步物理仿真里
+         通过轮地接触点的摩擦力反馈到车身上——而 VelocityControl 只接管了车身的
+         线速度/角速度(vx,vy,yaw角速度)这三个自由度，并不接管 z 高度和 roll/pitch，
+         这三个"没人管"的自由度会持续吸收这部分冲突产生的力矩，日积月累就是实测看到的
+         现象：机器人明明没怎么移动（长时间原地小范围巡游/自转），也没有撞到任何货架，
+         z 高度和俯仰角却在几十秒到一两分钟内缓慢爬升，最终以一个不上不下、卡住不动的
+         倾斜姿态"定住"。
+         根治办法：既然车身位移已经完全交给 VelocityControl 负责，轮子和地面之间就
+         不应该再有任何真实摩擦力参与——把 mu1/mu2 直接清零，轮子只保留碰撞形状用来
+         防止穿模，不再通过摩擦对车身产生任何反作用力，MecanumDrive 算出来的轮速只用来
+         让轮子在视觉上"转起来"，不变成任何实际作用力。这样两个插件才是真正互不干扰。 -->
     <gazebo reference="wheel_RF_Link">
-      <mu1>1.0</mu1>
-      <mu2>1.0</mu2>
+      <mu1>0.0</mu1>
+      <mu2>0.0</mu2>
     </gazebo>
     <gazebo reference="wheel_LF_Link">
-      <mu1>1.0</mu1>
-      <mu2>1.0</mu2>
+      <mu1>0.0</mu1>
+      <mu2>0.0</mu2>
     </gazebo>
     <gazebo reference="wheel_RR_Link">
-      <mu1>1.0</mu1>
-      <mu2>1.0</mu2>
+      <mu1>0.0</mu1>
+      <mu2>0.0</mu2>
     </gazebo>
     <gazebo reference="wheel_LR_Link">
-      <mu1>1.0</mu1>
-      <mu2>1.0</mu2>
+      <mu1>0.0</mu1>
+      <mu2>0.0</mu2>
     </gazebo>
   </xacro:macro>

File: ws_robot/src/astribot_s1_description/urdf/astribot_s1_torso_wheel.xacro (robot description, xacro)
@@ -3,15 +3,22 @@
   文件用途：Astribot S1 底盘部分（麦克纳姆全向轮 x4 + 4 自由度升降躯干）。
   数据来源：astribot_config/robot_config/astribot_s1/model/astribot_whole_body_with_wheel.urdf
-  （link/joint 名称、惯性参数、几何尺寸与原文件完全一致，未改动任何数值），本文件只做了两处必要修正：
+  （link/joint 名称、惯性参数、几何尺寸与原文件完全一致，未改动任何数值），本文件做了三处必要修正：
     1. mesh filename 由原文件里残缺的相对路径 "s1_torso/xxx.STL"
        改写为 package:// 形式，指向本包 CMakeLists.txt 安装的 meshes 目录；
     2. 四个轮子（wheel_RF/LF/RR/LR_Link）原文件完全没有 <collision>，仿真中会直接穿透地板，
-       这里按照实测 STL 包围盒（半径 0.08m、厚度 0.05m，见 config/collision_overrides.yaml）
-       补上圆柱体碰撞体 —— 对应任务书中"机器人生成后下坠/穿透地面"异常场景的修复。
+       这里按照实测 STL 包围盒（半径 0.08m）补上碰撞体 —— 对应任务书中
+       "机器人生成后下坠/穿透地面"异常场景的修复；
+    3. !!! 实测踩坑记录 !!!：碰撞体形状从圆柱改成了球体。起因是麦克纳姆轮平移 bug——
+       用官方 gz-sim 各向异性摩擦(fdir1+mu2=0)方案让轮子真正产生平移前，
+       对照 `/usr/share/ignition/ignition-gazebo6/worlds/mecanum_drive.sdf`
+       官方示例发现它的轮子碰撞体用的是球体而不是圆柱体。球体在任意姿态下都是干净的
+       单点接触，圆柱在轮子侧滚接触时理论上也是单点接触，但数值上更容易在边缘/端面出现
+       意外的多点/线接触导致摩擦方向解算不稳定——球体更贴合"各向异性摩擦只在一个干净
+       接触点上生效"这个假设，改成球体后经实测确认轮子真的能带动底盘平移了
+       （见 astribot_s1.gazebo.xacro 里 fdir1/mu2 配置的详细说明）。
 -->
 <robot xmlns:xacro="http://www.ros.org/wiki/xacro">
   <!-- 麦克纳姆轮碰撞体公共尺寸（来自 STL 包围盒实测，见 config/collision_overrides.yaml） -->
   <xacro:property name="wheel_collision_radius" value="0.08"/>
-  <xacro:property name="wheel_collision_length" value="0.05"/>
   <!-- 躯干底座：唯一根 link，无 parent；平动升降+轮式全向底盘均挂在它上面 -->
   <link name="astribot_torso_base">
@@ -53,9 +60,11 @@
       </material>
     </visual>
-    <!-- 补充碰撞体：圆柱沿 link 局部 Z 轴（即转轴）——原文件缺失，必须补，否则轮子会穿地 -->
-    <collision>
-      <origin rpy="0 0 0" xyz="0 0 0.0145"/>
-      <geometry>
-        <cylinder radius="${wheel_collision_radius}" length="${wheel_collision_length}"/>
+    <!-- 补充碰撞体：球体，中心与轮子局部原点重合——原文件缺失，必须补，否则轮子会穿地；
+         用球体而不是圆柱体是为了配合麦克纳姆轮各向异性摩擦(fdir1/mu2)方案，
+         见文件顶部注释第3点和 astribot_s1.gazebo.xacro 里的详细说明 -->
+    <collision>
+      <origin rpy="0 0 0" xyz="0 0 0.0145"/>
+      <geometry>
+        <sphere radius="${wheel_collision_radius}"/>
       </geometry>
     </collision>
@@ -85,5 +94,5 @@
       <origin rpy="0 0 0" xyz="0 0 0.0145"/>
       <geometry>
-        <cylinder radius="${wheel_collision_radius}" length="${wheel_collision_length}"/>
+        <sphere radius="${wheel_collision_radius}"/>
       </geometry>
     </collision>
@@ -113,5 +122,5 @@
       <origin rpy="0 0 0" xyz="0 0 0.0145"/>
       <geometry>
-        <cylinder radius="${wheel_collision_radius}" length="${wheel_collision_length}"/>
+        <sphere radius="${wheel_collision_radius}"/>
       </geometry>
     </collision>
@@ -141,5 +150,5 @@
       <origin rpy="0 0 0" xyz="0 0 0.0145"/>
       <geometry>
-        <cylinder radius="${wheel_collision_radius}" length="${wheel_collision_length}"/>
+        <sphere radius="${wheel_collision_radius}"/>
       </geometry>
     </collision>
