Commit message: 移除双运动学插件，车轮改用 effort 力矩接口
原架构同时挂着两套互不相关的运动学：VelocityControl 直接改写
base_link 的本体速度（完全绕过轮地接触力），MecanumDrive 另外
独立驱动四个轮关节（纯视觉效果）。车身运动和车轮转动之间没有任何
力学耦合，所以既无法复现真实的摩擦/打滑行为，也没有任何力学纠错
机制去抵消侧向偏差——这是长期倾倒问题的架构性根因。

改造内容：
- astribot_s1.gazebo.xacro: 删除 VelocityControl 和 MecanumDrive 两个
  system 插件（保留 OdometryPublisher/Sensors），恢复四轮各向异性摩擦
  SDF 配置，注释里保留第一至四轮踩坑记录备查
- astribot_s1_ros2_control.xacro: 四个轮关节接入 effort command_interface
  + position/velocity/effort state_interface
- astribot_s1_torso_wheel.xacro: 轮碰撞半径参数化为 $(arg wheel_radius)；
  四个轮关节补上 <limit> 和 <dynamics damping/friction>——原文件两者
  皆无，轮子是几乎无阻尼的自由旋转体(izz=0.0015639)，力矩闭环下会在
  几毫秒内被加速到速度限位并在扭矩限幅之间 bang-bang 振荡
- astribot_s1_controllers.yaml: 新增 wheel_effort_controller
  (forward_command_controller, interface_name: effort)，并把四个轮关节
  加进 joint_state_broadcaster 的 joints 白名单

两个实测踩坑，都记在对应文件的注释里：
1. effort command_interface 内写 <param name="min"/>/<param name="max"/>
   （官方文档形式）会让 gz_ros2_control 静默跳过整个关节，日志里连
   "Loading joint:" 都没有，激活时报 "Not acceptable command interfaces
   combination"。实测环境 hardware-interface 2.54.0 + gz-ros2-control
   0.7.20 只接受裸标签，限幅改在上层节点做。
2. joint_state_broadcaster 的 joints 白名单漏掉轮关节，会让上层看到
   永久过期的反馈、失效保护一直把力矩压在 0，症状和接口没加载一模一样。

已知限制：dartsim 不调用 setSecondaryFrictionCoeff（nm -D -u 符号确认），
SDF 里的 mu2 实际被忽略，拿不到真正的横向自由滑动，等效为各向同性摩擦。

Co-Authored-By: Claude <noreply@anthropic.com>

File: ws_robot/src/astribot_s1_description/urdf/astribot_s1.gazebo.xacro (robot description, xacro)
@@ -12,8 +12,8 @@
 -->
 <robot xmlns:xacro="http://www.ros.org/wiki/xacro">
-  <xacro:macro name="astribot_s1_gazebo_chassis_plugins"
-               params="robot_name:=astribot_s1 wheel_radius:=0.08 wheel_separation:=0.4327 wheelbase:=0.4327">
-    <!-- ========== 底盘全向驱动：VelocityControl(实际驱动身体位移) + MecanumDrive(轮子视觉旋转) ==========
-         !!! 实测踩坑记录（麦克纳姆轮"轮子转、车不走"bug 的完整排查过程）!!!
+  <xacro:macro name="astribot_s1_gazebo_chassis_plugins" params="robot_name:=astribot_s1">
+    <!-- ========== 底盘驱动架构演进史（麦克纳姆轮"轮子转、车不走"→"两套独立运动学
+         打架诱发倾倒"→"治本：力矩闭环"的完整排查过程，务必先读完再改这个文件）==========
+         !!! 实测踩坑记录 !!!
          第一轮尝试：给四个轮子配置各向异性摩擦（fdir1 按 45°对角线 + mu2=0，完全照抄
          gz-sim 官方示例 `/usr/share/ignition/ignition-gazebo6/worlds/mecanum_drive.sdf`
@@ -26,50 +26,36 @@
              不是文档记录的已知限制，是本方案实测发现的）。本机器人轮子半径只有0.08m，
              正好落在这个失效区间内，所以无论怎么调摩擦系数/坐标系表达都不会有效果。
-         第二轮修复（本方案最终采用）：改用 gz-sim 官方 `VelocityControl` 系统插件
-         （示例：`/usr/share/ignition/ignition-gazebo6/worlds/velocity_control.sdf`）
-         ——它不依赖轮子-地面摩擦力学，而是直接对模型本体设置线速度/角速度，
-         从根本上绕开了"小尺寸轮子摩擦近似失效"这个物理引擎数值问题，实测在本机器人
-         真实质量(39kg躯干)和真实轮子尺寸(0.08m)下 x/y/yaw 三个自由度平移旋转都正常。
-         MecanumDrive 插件保留下来，只用来让轮子按论理转速转起来做视觉效果
-         （它自己单独驱动的车身位移量在我们的尺寸下可忽略不计，不会和 VelocityControl
-         的真实位移打架，两者互不干扰，同时生效）。 -->
+         第二轮修复：改用 gz-sim 官方 `VelocityControl` 系统插件直接对模型本体设置
+         线速度/角速度，绕开"小尺寸轮子摩擦近似失效"问题，配合 `MecanumDrive` 插件
+         单独驱动四个轮子关节做视觉转动——这是很长一段时间的"最终采用"方案。
+         第三轮踩坑（真正的"平移正常但会慢慢倾倒"根因）：MecanumDrive 独立按运动学
+         公式算轮速、VelocityControl 独立设定车身速度，两者互不知情；只要轮子还有
+         摩擦(mu1/mu2>0)，两套独立计算的残差就会通过轮地接触点反馈到车身，而
+         VelocityControl 不接管 z/roll/pitch，这三个自由度持续吸收残差力矩，
+         日积月累导致"没撞任何东西也会缓慢倾倒"。根治：把 mu1/mu2 直接清零。
+         第四轮尝试（已实测验证不可行，已回退）：想在清零摩擦的基础上重新引入一组
+         大幅收紧的各向异性摩擦，做"可量化误差力矩风险"和"真实轮地约束"之间的折中。
+         4组测试（纯旋转零漂移 vs 纯平移必然复现倾倒，且跟mu大小无关只跟时长/路程
+         相关）证实：只要 MecanumDrive+VelocityControl 两套独立运动学并行的架构不变，
+         mu>0 就必然有风险，不是参数问题，是结构问题——真正的根治方案只能是把两套
+         独立运动学合并成一条经过真实轮地接触物理的力矩闭环链路。
+         !!! 第五轮（治本改造，本次落地）!!!：按"麦轮力控重构方案"实施——
+           - VelocityControl、MecanumDrive 两个插件**整体移除**（见下方，不再声明）；
+           - 车身运动完全由轮子 effort 力矩经真实轮地接触摩擦驱动，力矩由新增的
+             astribot_s1_chassis_effort_drive 包（mecanum_effort_drive_node：
+             麦克纳姆逆解 + 轮速PID + 摩擦前馈）计算，经 ros2_control 的
+             effort command_interface 下发（见 astribot_s1_ros2_control.xacro）；
+           - 车轮不再需要"视觉转动"这个概念——转速是真实力矩驱动出来的物理结果，
+             跟车身位移天然一致，不存在"两套独立运动学"这个问题了；
+           - 各向异性摩擦（fdir1对角线方案，第一轮已验证的坐标系表达）重新启用，
+             但语义变了：mu 不再是"尽量清零避免冲突残差"，是**真实驱动摩擦力**，
+             第一轮"小轮子在DART下数值不稳定"这个历史踩坑依然可能复现——如果这次
+             实测又出现"轮转车不动"，先跑接触求解器调参清单，再考虑TPE物理引擎，
+             不要立刻怀疑逆解代码，两种故障现象不同（符号错了是"转向不对/原地
+             打转"，摩擦失效是"轮子转但完全没有对应位移"）。 -->
     <gazebo>
-      <plugin filename="gz-sim-velocity-control-system" name="gz::sim::systems::VelocityControl">
-        <!-- 兼容提示：ignition-gazebo-velocity-control-system /
-             ignition::gazebo::systems::VelocityControl。
-             没有 <topic> 子标签可配置——它固定订阅 "/model/<模型名>/cmd_vel"
-             （官方示例验证过，和 ros_gz_bridge 里桥接的目标话题名天然一致，不用额外配置）。 -->
-      </plugin>
-      <plugin filename="gz-sim-mecanum-drive-system" name="gz::sim::systems::MecanumDrive">
-        <!-- 兼容提示（旧版 Ignition Gazebo Fortress 早期/自编译环境可能仍需要这两行写法）：
-             filename="ignition-gazebo-mecanum-drive-system"
-             name="ignition::gazebo::systems::MecanumDrive" -->
-        <front_left_joint>wheel_LF_Joint</front_left_joint>
-        <front_right_joint>wheel_RF_Joint</front_right_joint>
-        <back_left_joint>wheel_LR_Joint</back_left_joint>
-        <back_right_joint>wheel_RR_Joint</back_right_joint>
-        <wheel_separation>${wheel_separation}</wheel_separation>
-        <wheelbase>${wheelbase}</wheelbase>
-        <wheel_radius>${wheel_radius}</wheel_radius>
-        <!-- 与 astribot_chassis.yaml 的 joint_max_velocities: [1.0, 1.0, 2.0] (x, y, yaw) 保持一致 -->
-        <max_linear_velocity>1.0</max_linear_velocity>
-        <min_linear_velocity>-1.0</min_linear_velocity>
-        <max_angular_velocity>2.0</max_angular_velocity>
-        <min_angular_velocity>-2.0</min_angular_velocity>
-        <min_acceleration>-5.0</min_acceleration>
-        <max_acceleration>5.0</max_acceleration>
-        <min_jerk>-50.0</min_jerk>
-        <max_jerk>50.0</max_jerk>
-        <!-- !!! 实测踩坑记录 !!!：MecanumDrive 的 <topic> 只要显式写了，就是"字面量"话题名，
-             不会像 OdometryPublisher 的 <odom_topic> 那样自动补上 "/model/<name>/" 前缀，
-             必须显式写成和 ros_gz_bridge 配置一致的绝对话题名，否则订阅不到消息。 -->
-        <topic>/model/${robot_name}/cmd_vel</topic>
-        <odom_topic>/model/${robot_name}/mecanum_odometry</odom_topic>
-        <frame_id>odom</frame_id>
-        <child_frame_id>astribot_torso_base</child_frame_id>
-      </plugin>
       <!-- MecanumDrive/VelocityControl 都不发布可靠的 TF，单独挂 OdometryPublisher 补
-           /tf 与 nav_msgs/Odometry（它是基于模型真实位姿变化算出来的，不受上面选用哪个
-           驱动插件影响）。
+           /tf 与 nav_msgs/Odometry（它是基于模型真实位姿变化算出来的，跟底盘是运动学
+           直控还是力矩闭环驱动完全无关，两套架构切换都不用碰这个插件）。
            !!! 实测踩坑记录 !!!：一开始仿照 MecanumDrive 那样给它加了显式的
            <odom_topic>/<tf_topic> 绝对路径，结果这个插件直接不再发布任何东西了
@@ -86,12 +72,12 @@
         <dimensions>3</dimensions>
       </plugin>
-      <!-- !!! 实测踩坑记录（新增，非常关键）!!!：aws_robomaker_small_warehouse_world 的
+      <!-- !!! 实测踩坑记录（非常关键）!!!：aws_robomaker_small_warehouse_world 的
            world 文件本身一个 <plugin> 标签都没有，gz-sim 找不到 world 级插件配置时，
            会退回 ~/.gz(或.ignition)/sim/<ver>/server.config 里的默认系统插件列表——
            实测那份默认列表只有 Physics/UserCommands/SceneBroadcaster 三个，
            **没有 Sensors 系统**！缺了它，机器人身上所有 camera/gpu_lidar 传感器
-           （包括这里新加的双 Livox Mid-360，也包括头部相机）只会被解析、
-           永远不会真正渲染/发布任何数据——话题能在 `ros2 topic list` 里看到，
-           但 `ros2 topic hz` 永远拿不到消息，很容易被误判成"话题名/桥接配置错了"。
+           （包括双 Livox Mid-360，也包括头部相机）只会被解析、永远不会真正渲染/
+           发布任何数据——话题能在 `ros2 topic list` 里看到，但 `ros2 topic hz`
+           永远拿不到消息，很容易被误判成"话题名/桥接配置错了"。
            因为不允许修改 aws 官方仓库的 world 文件，这里改成把 Sensors 系统插件挂在
            "我们自己机器人模型"的 <gazebo> 标签下——gz-sim 的 Sensors 系统一旦在
@@ -103,38 +89,123 @@
       </plugin>
     </gazebo>
-    <!-- !!! 实测踩坑记录（第三轮，真正的"平移正常但会慢慢倾倒"根因）!!!：上一版本把
-         四个轮子摩擦系数恢复成普通各向同性摩擦(mu1=mu2=1.0)，理由是"轮子不再负责实际
-         驱动身体位移，只是给轮子一个合理的地面摩擦力，避免打滑的观感问题"——这个理由
-         本身是错的。MecanumDrive 插件仍然在**独立**按照它自己内部的全向轮运动学公式
-         计算并驱动四个轮子关节的转速（只是为了让轮子在视觉上转得"看起来对"），这个转速
-         是按"轮子和地面之间存在真实摩擦、靠摩擦力驱动车身"这个假设算出来的；但车身实际
-         的位移是由 VelocityControl 直接设定的，和轮子转速隐含的"应有位移"并不是同一回事
-         （两者独立计算，几乎不可能完全一致）。只要轮子还有摩擦(mu1/mu2>0)，这个"轮子
-         转速暗示的运动"和"车身实际被强制的运动"之间的差异，就会在每一步物理仿真里
-         通过轮地接触点的摩擦力反馈到车身上——而 VelocityControl 只接管了车身的
-         线速度/角速度(vx,vy,yaw角速度)这三个自由度，并不接管 z 高度和 roll/pitch，
-         这三个"没人管"的自由度会持续吸收这部分冲突产生的力矩，日积月累就是实测看到的
-         现象：机器人明明没怎么移动（长时间原地小范围巡游/自转），也没有撞到任何货架，
-         z 高度和俯仰角却在几十秒到一两分钟内缓慢爬升，最终以一个不上不下、卡住不动的
-         倾斜姿态"定住"。
-         根治办法：既然车身位移已经完全交给 VelocityControl 负责，轮子和地面之间就
-         不应该再有任何真实摩擦力参与——把 mu1/mu2 直接清零，轮子只保留碰撞形状用来
-         防止穿模，不再通过摩擦对车身产生任何反作用力，MecanumDrive 算出来的轮速只用来
-         让轮子在视觉上"转起来"，不变成任何实际作用力。这样两个插件才是真正互不干扰。 -->
+    <!-- !!! 各向异性摩擦：真实驱动力，不是第四轮的"误差力矩折中"（第五轮/治本改造） !!!
+         力矩闭环架构下，摩擦力是轮子唯一的驱动力来源，mu 从第四轮的收紧值(0.05)
+         改回接近真实橡胶轮-混凝土地面实测范围(0.6~0.8)，比第一轮用过的1.0略低作为
+         起点。collision 命名沿用离线核对过的 "<link名>_collision" 正确格式。
+         fdir1 方向沿用第一轮验证过的对角线模式(RF/LR共享一条对角线、LF/RR共享另一条)，
+         ignition:expressed_in="astribot_torso_base" 写法也是第一轮验证过的，直接复用。
+         kp/kd 比第四轮更硬(1e6/50 vs 1e5/10)：第四轮软化是为了减少"运动学冲突残差"
+         的接触抖动，现在不存在这个冲突了，需要的是真实支撑力，配置太软容易穿透。
+         这组 mu/kp/kd 都是起始估算值，未经实测标定，部署前必须先跑方案第8节的
+         分级测试①②③，尤其关注第一轮记录过的"小轮子在DART下数值不稳定"是否复现——
+         如果复现，先走接触求解器调参清单，这也是本次"改变轮子大小做多轮测试"重点
+         要验证的问题：数值不稳定的边界到底在多大的轮径。 -->
     <gazebo reference="wheel_RF_Link">
-      <mu1>0.0</mu1>
-      <mu2>0.0</mu2>
+      <collision name="wheel_RF_Link_collision">
+        <surface>
+          <friction>
+            <ode>
+              <mu>0.7</mu>
+              <mu2>0.0</mu2>
+              <fdir1 xmlns:ignition="http://ignitionrobotics.org/schema"
+                     ignition:expressed_in="astribot_torso_base">1 1 0</fdir1>
+            </ode>
+            <torsional>
+              <coefficient>0.05</coefficient>
+              <use_patch_radius>true</use_patch_radius>
+              <patch_radius>0.01</patch_radius>
+            </torsional>
+          </friction>
+          <contact>
+            <ode>
+              <kp>1e6</kp>
+              <kd>50.0</kd>
+              <max_vel>0.05</max_vel>
+              <min_depth>0.0005</min_depth>
+            </ode>
+          </contact>
+        </surface>
+      </collision>
     </gazebo>
     <gazebo reference="wheel_LF_Link">
-      <mu1>0.0</mu1>
-      <mu2>0.0</mu2>
+      <collision name="wheel_LF_Link_collision">
+        <surface>
+          <friction>
+            <ode>
+              <mu>0.7</mu>
+              <mu2>0.0</mu2>
+              <fdir1 xmlns:ignition="http://ignitionrobotics.org/schema"
+                     ignition:expressed_in="astribot_torso_base">1 -1 0</fdir1>
+            </ode>
+            <torsional>
+              <coefficient>0.05</coefficient>
+              <use_patch_radius>true</use_patch_radius>
+              <patch_radius>0.01</patch_radius>
+            </torsional>
+          </friction>
+          <contact>
+            <ode>
+              <kp>1e6</kp>
+              <kd>50.0</kd>
+              <max_vel>0.05</max_vel>
+              <min_depth>0.0005</min_depth>
+            </ode>
+          </contact>
+        </surface>
+      </collision>
     </gazebo>
     <gazebo reference="wheel_RR_Link">
-      <mu1>0.0</mu1>
-      <mu2>0.0</mu2>
+      <collision name="wheel_RR_Link_collision">
+        <surface>
+          <friction>
+            <ode>
+              <mu>0.7</mu>
+              <mu2>0.0</mu2>
+              <fdir1 xmlns:ignition="http://ignitionrobotics.org/schema"
+                     ignition:expressed_in="astribot_torso_base">1 -1 0</fdir1>
+            </ode>
+            <torsional>
+              <coefficient>0.05</coefficient>
+              <use_patch_radius>true</use_patch_radius>
+              <patch_radius>0.01</patch_radius>
+            </torsional>
+          </friction>
+          <contact>
+            <ode>
+              <kp>1e6</kp>
+              <kd>50.0</kd>
+              <max_vel>0.05</max_vel>
+              <min_depth>0.0005</min_depth>
+            </ode>
+          </contact>
+        </surface>
+      </collision>
     </gazebo>
     <gazebo reference="wheel_LR_Link">
-      <mu1>0.0</mu1>
-      <mu2>0.0</mu2>
+      <collision name="wheel_LR_Link_collision">
+        <surface>
+          <friction>
+            <ode>
+              <mu>0.7</mu>
+              <mu2>0.0</mu2>
+              <fdir1 xmlns:ignition="http://ignitionrobotics.org/schema"
+                     ignition:expressed_in="astribot_torso_base">1 1 0</fdir1>
+            </ode>
+            <torsional>
+              <coefficient>0.05</coefficient>
+              <use_patch_radius>true</use_patch_radius>
+              <patch_radius>0.01</patch_radius>
+            </torsional>
+          </friction>
+          <contact>
+            <ode>
+              <kp>1e6</kp>
+              <kd>50.0</kd>
+              <max_vel>0.05</max_vel>
+              <min_depth>0.0005</min_depth>
+            </ode>
+          </contact>
+        </surface>
+      </collision>
     </gazebo>
   </xacro:macro>

File: ws_robot/src/astribot_s1_description/urdf/astribot_s1.xacro (robot description, xacro)
@@ -28,4 +28,23 @@
        本文件内部不出现任何硬编码路径。 -->
   <xacro:arg name="controllers_config" default=""/>
+  <!-- 麦克纳姆轮力矩闭环驱动改造新增：轮子effort硬件接口边界 + 几何半径统一从这里
+       外部传入，禁止在 torso_wheel/ros2_control xacro 里写死。
+       wheel_radius 同时驱动碰撞体球半径(astribot_s1_torso_wheel.xacro)和
+       astribot_s1_chassis_effort_drive 包里逆解运动学的同名ROS2参数——
+       "改变轮子大小做多轮测试"时只需要改这一个xacro参数，但 spawn_z 要跟着按
+       spawn_z=0.02+wheel_radius 这个经验公式同步调整(见
+       astribot_s1_gazebo_bringup/launch/warehouse_sim.launch.py 的 spawn_z 说明)，
+       否则出生时轮子和地面的穿透/悬空量不对，扫描结果没有意义。
+       wheel_effort_limit/wheel_velocity_limit 是轮关节URDF<limit>标签和
+       ros2_control effort command_interface的min/max边界，起始估算值，
+       需要方案里的单轮测试①标定。 -->
+  <xacro:arg name="wheel_radius" default="0.08"/>
+  <xacro:arg name="wheel_effort_limit" default="15.0"/>
+  <xacro:arg name="wheel_velocity_limit" default="40.0"/>
+  <!-- 轮关节粘性阻尼(N·m·s/rad)和静摩擦(N·m)：力矩闭环稳定的必要条件，
+       没有它轮子是无阻尼自由旋转体、PID会在扭矩限幅间bang-bang振荡，
+       详见 astribot_s1_torso_wheel.xacro 顶部"轮关节dynamics"实测记录。 -->
+  <xacro:arg name="wheel_joint_damping" default="1.0"/>
+  <xacro:arg name="wheel_joint_friction" default="0.1"/>
   <xacro:property name="use_lidar_prop" value="$(arg use_lidar)"/>
   <xacro:property name="use_camera_prop" value="$(arg use_camera)"/>
@@ -53,7 +72,16 @@
   </xacro:if>
   <!-- ============ ros2_control + gz_ros2_control 插件 ============ -->
+  <!-- wheel_effort_limit 不再传进 astribot_s1_ros2_control 宏——实测发现
+       gz_ros2_control(ros-humble-hardware-interface 2.54.0) 解析
+       <command_interface name="effort"><param name="min"/><param name="max"/></command_interface>
+       这种带子标签的写法时会把该关节整体跳过(initSim日志里"Loading joint"
+       完全不出现)，改成最简单的<command_interface name="effort"/>后正常。
+       力矩限幅改成完全交给 astribot_s1_chassis_effort_drive 包的PID闭环代码
+       clamp(软件层强制限幅，真正生效的那一层)，详见
+       astribot_s1_ros2_control.xacro 里的踩坑记录。 -->
   <xacro:astribot_s1_ros2_control controllers_config="$(arg controllers_config)"/>
-  <!-- ============ 底盘全向轮驱动 + 里程计 + 轮子摩擦 ============ -->
-  <xacro:astribot_s1_gazebo_chassis_plugins
-    robot_name="${robot_name_prop}" wheel_radius="0.08" wheel_separation="0.4327" wheelbase="0.4327"/>
+  <!-- ============ 底盘：里程计发布 + 轮子各向异性摩擦(力矩闭环治本改造后，
+       VelocityControl/MecanumDrive 已移除，车身运动完全由轮子effort力矩经
+       轮地接触物理驱动，见 astribot_s1_chassis_effort_drive 包) ============ -->
+  <xacro:astribot_s1_gazebo_chassis_plugins robot_name="${robot_name_prop}"/>
 </robot>

File: ws_robot/src/astribot_s1_description/urdf/astribot_s1_ros2_control.xacro (robot description, xacro)
@@ -3,10 +3,18 @@
   文件用途：为躯干升降(4)+头部(2)+左臂(7)+右臂(7) 共 20 个 revolute 关节声明 <ros2_control> 硬件接口，
   并挂载 gz_ros2_control 的 Gazebo 系统插件，使 ros2_control 的 controller_manager 能在 gz sim 内部运行。
-  注意：4 个轮子(wheel_*_Joint) 不在这里声明，底盘运动学由 astribot_s1.gazebo.xacro 里的
-  MecanumDrive 系统插件直接接管（原生支持全向运动，无需再套 ros2_control），
-  避免"同一关节被两个控制系统同时下发指令"的冲突。
+  !!! 麦轮力控重构方案实施记录（治本改造）!!!：4 个轮子(wheel_*_Joint) 原来不在这里声明，
+  理由是"底盘运动学由 astribot_s1.gazebo.xacro 里的 MecanumDrive 系统插件直接接管，
+  避免同一关节被两个控制系统同时下发指令的冲突"——现在 MecanumDrive 和 VelocityControl
+  两个插件已经整体移除（见 astribot_s1.gazebo.xacro 的对应记录），轮子改成通过
+  effort command_interface 接入 ros2_control，由 astribot_s1_chassis_effort_drive 包的
+  mecanum_effort_drive_node 计算力矩、经 forward_command_controller 下发，不再有
+  "两个控制系统抢同一个关节"这个问题——这正是本次改造要消除的东西，现在轮子和
+  躯干/头部/双臂共用同一个 ros2_control 硬件实例、同一个 controller_manager，
+  是治本方案的一部分，不是疏忽。
   command_interface 统一用 position（对应真实设备的位置控制模式，也是 astribot_*.yaml 里
   frequency/coefficient 抽象所隐含的控制方式）；state_interface 同时给 position+velocity，
-  供 joint_state_broadcaster 发布完整 /joint_states。
+  供 joint_state_broadcaster 发布完整 /joint_states。轮子单独用 effort command_interface
+  （见下面 astribot_s1_effort_wheel_joint 宏），跟其它20个position关节类型不同但
+  ros2_control 原生支持同一硬件实例内混用不同 command_interface 类型。
 -->
 <robot xmlns:xacro="http://www.ros.org/wiki/xacro">
@@ -14,4 +22,28 @@
     <joint name="${name}">
       <command_interface name="position"/>
+      <state_interface name="position"/>
+      <state_interface name="velocity"/>
+      <state_interface name="effort"/>
+    </joint>
+  </xacro:macro>
+  <!-- 轮子effort硬件接口。
+       !!! 实测踩坑记录(本次任务新增)!!!：最初按 gz_ros2_control 官方文档示例写法，
+       在 <command_interface name="effort"> 下加了 <param name="min">/<param name="max">
+       子标签做min/max边界声明——结果实测这4个轮关节被 gz_ros2_control 的
+       initSim **整体跳过**：启动日志里只有"Loading joint: astribot_xxx"20条
+       (躯干/头部/双臂，全部是不带<param>子标签的position接口)，wheel_*_Joint
+       一条都没出现，导致 export_command_interfaces 里根本不存在这4个effort接口，
+       controller_manager激活wheel_effort_controller时报"Not existing"直接拒绝。
+       躯干/头部/双臂的20个关节写法完全不带<param>子标签、正常加载，只有带
+       <param>子标签的这4个轮关节被跳过——两者唯一差异就是这个<param>子标签，
+       实测确认是这个版本(ros-humble-hardware-interface 2.54.0)的URDF解析在
+       command_interface带子标签时有问题。既然效力限幅本来就在
+       astribot_s1_chassis_effort_drive包的PID闭环里做了强制clamp(软件层，
+       真正生效的那一层)，这里的<param>只是"补充声明"，不是必须的，直接去掉，
+       只留最简单的 <command_interface name="effort"/>，跟20个position关节
+       的写法保持同样"干净"的格式。 -->
+  <xacro:macro name="astribot_s1_effort_wheel_joint" params="name">
+    <joint name="${name}">
+      <command_interface name="effort"/>
       <state_interface name="position"/>
       <state_interface name="velocity"/>
@@ -46,4 +78,8 @@
       <xacro:astribot_s1_position_joint name="astribot_arm_right_joint_6"/>
       <xacro:astribot_s1_position_joint name="astribot_arm_right_joint_7"/>
+      <xacro:astribot_s1_effort_wheel_joint name="wheel_RF_Joint"/>
+      <xacro:astribot_s1_effort_wheel_joint name="wheel_LF_Joint"/>
+      <xacro:astribot_s1_effort_wheel_joint name="wheel_RR_Joint"/>
+      <xacro:astribot_s1_effort_wheel_joint name="wheel_LR_Joint"/>
     </ros2_control>
     <gazebo>

File: ws_robot/src/astribot_s1_description/urdf/astribot_s1_torso_wheel.xacro (robot description, xacro)
@@ -19,6 +19,11 @@
 -->
 <robot xmlns:xacro="http://www.ros.org/wiki/xacro">
-  <!-- 麦克纳姆轮碰撞体公共尺寸（来自 STL 包围盒实测，见 config/collision_overrides.yaml） -->
-  <xacro:property name="wheel_collision_radius" value="0.08"/>
+  <!-- 麦克纳姆轮碰撞体公共尺寸——治本改造后改成从顶层 astribot_s1.xacro 的
+       $(arg wheel_radius) 传入(默认仍是0.08m，跟原STL包围盒实测值一致)，
+       不再写死，专门为"改变轮子大小做多轮测试"这个扫描场景准备。
+       改这个值只影响碰撞球半径本身，轮子关节origin/spawn_z等其它几何量
+       不会跟着自动联动，扫描测试前必须按 astribot_s1_chassis_effort_drive/
+       README_CHASSIS_EFFORT_DRIVE.md 里的公式手动同步调整spawn_z。 -->
+  <xacro:property name="wheel_collision_radius" value="$(arg wheel_radius)"/>
   <!-- 躯干底座：唯一根 link，无 parent；平动升降+轮式全向底盘均挂在它上面 -->
   <link name="astribot_torso_base">
@@ -60,5 +65,21 @@
     </collision>
   </link>
-  <!-- ============ 四个麦克纳姆轮（各自朝向旋转45°/135°，构成全向底盘） ============ -->
+  <!-- ============ 四个麦克纳姆轮（各自朝向旋转45°/135°，构成全向底盘） ============
+       !!! 轮关节 dynamics(阻尼/静摩擦) 实测记录（力控重构方案新增）!!!：
+       原文件四个轮关节既没有<limit>也没有<dynamics>，轮子在物理上是一个几乎
+       "无阻尼自由旋转体"(izz只有0.0015639 kg·m²)。切到 effort 力矩闭环之后
+       实测暴露出问题：只要地面反作用力不足(实测是逆解系数配错导致四轮力矩
+       互相抵消)，轮子会在几毫秒内被力矩加速到关节速度限位(±40rad/s)，
+       PID随即看到巨大误差、把力矩打到反向限幅，来回bang-bang剧烈振荡，
+       转速在±40之间跳变完全不收敛。真实带减速器的轮驱动本身就存在可观的
+       粘性阻尼和静摩擦，补上 <dynamics damping/friction> 既是物理保真，
+       也是力矩闭环能稳定收敛的必要条件。两个值都走xacro参数，便于按实测调整。
+       !!! 另一个重要的几何事实（逆解必须按这个来）!!!：下面四个轮关节的
+       origin rpy 决定了轮子**轴线在torso_base系里指向45°对角线**
+       (RF=[0.707,-0.707,0]、LF=[0.707,0.707,0]、RR=[-0.707,-0.707,0]、
+       LR=[-0.707,0.707,0])——这是一台 **X型布局全向轮(omni)** 底盘，
+       不是"轮轴沿±y、辊子45°"的标准麦克纳姆布局，两者的运动学逆解公式完全
+       不同。逆解系数推导见 astribot_s1_chassis_effort_drive/config/
+       mecanum_effort_drive_params.yaml 顶部注释。 -->
   <link name="wheel_RF_Link">
     <inertial>
@@ -91,4 +112,12 @@
     <child link="wheel_RF_Link"/>
     <axis xyz="0 0 1"/>
+    <!-- 力控重构方案新增：原文件里continuous轮关节完全没有limit标签(实测确认，
+         对比躯干关节都有effort/velocity)。effort/velocity边界从顶层xacro:arg
+         传入，须跟astribot_s1_ros2_control.xacro的effort command_interface
+         min/max、astribot_s1_chassis_effort_drive的wheel_effort_limit_nm
+         参数保持同一个数值。 -->
+    <limit effort="$(arg wheel_effort_limit)" velocity="$(arg wheel_velocity_limit)"/>
+    <!-- 关节阻尼/静摩擦：力控闭环稳定的必要条件，详见本文件顶部"轮关节dynamics"说明 -->
+    <dynamics damping="$(arg wheel_joint_damping)" friction="$(arg wheel_joint_friction)"/>
   </joint>
   <link name="wheel_LF_Link">
@@ -119,4 +148,7 @@
     <child link="wheel_LF_Link"/>
     <axis xyz="0 0 1"/>
+    <limit effort="$(arg wheel_effort_limit)" velocity="$(arg wheel_velocity_limit)"/>
+    <!-- 关节阻尼/静摩擦：力控闭环稳定的必要条件，详见本文件顶部"轮关节dynamics"说明 -->
+    <dynamics damping="$(arg wheel_joint_damping)" friction="$(arg wheel_joint_friction)"/>
   </joint>
   <link name="wheel_RR_Link">
@@ -147,4 +179,7 @@
     <child link="wheel_RR_Link"/>
     <axis xyz="0 0 1"/>
+    <limit effort="$(arg wheel_effort_limit)" velocity="$(arg wheel_velocity_limit)"/>
+    <!-- 关节阻尼/静摩擦：力控闭环稳定的必要条件，详见本文件顶部"轮关节dynamics"说明 -->
+    <dynamics damping="$(arg wheel_joint_damping)" friction="$(arg wheel_joint_friction)"/>
   </joint>
   <link name="wheel_LR_Link">
@@ -175,4 +210,7 @@
     <child link="wheel_LR_Link"/>
     <axis xyz="0 0 1"/>
+    <limit effort="$(arg wheel_effort_limit)" velocity="$(arg wheel_velocity_limit)"/>
+    <!-- 关节阻尼/静摩擦：力控闭环稳定的必要条件，详见本文件顶部"轮关节dynamics"说明 -->
+    <dynamics damping="$(arg wheel_joint_damping)" friction="$(arg wheel_joint_friction)"/>
   </joint>
   <!-- ============ 4 自由度升降躯干（astribot_torso_joint_1..4） ============ -->
