Commit message: 同步工作树：自主探索退役重构、建图/搬运/社交导航/算子站新包与文档
- astribot_s1_autonomy 退役，逻辑并入 astribot_s1_exploration 与 astribot_autonomy_core
- 新增 map_manager / operator_station(+backend/msgs) / route_executor / transport(+mtc) / social_navigation / slam / robot_geometry / eigen_vendor 等包
- astribot_s1_navigation_msgs 增补 Envelope/Maneuver/Social/ArmHold 等 msg 与 srv
- astribot_s1_path_tracking / navigation_policy 增补 arrival、corridor、slip、social 等模块
- 补大量运行/验证文档、工具与测试脚本；.gitignore 忽略 runs/ 运行产物

Co-Authored-By: Claude Code <noreply@anthropic.com>

File: ws_robot/src/astribot_s1_description/urdf/astribot_s1.gazebo.xacro (robot description, xacro)
@@ -84,4 +84,5 @@
            场景里任意实体上加载成功，就会全局接管整个仿真里所有传感器的渲染，
            不需要非挂在 world 实体上不可，这是应对"不能改 world 文件"场景的标准做法。 -->
+      <plugin filename="ignition-gazebo-imu-system" name="gz::sim::systems::Imu"/>
       <plugin filename="gz-sim-sensors-system" name="gz::sim::systems::Sensors">
         <!-- 兼容提示：ignition-gazebo-sensors-system / ignition::gazebo::systems::Sensors -->

File: ws_robot/src/astribot_s1_description/urdf/astribot_s1.xacro (robot description, xacro)
@@ -15,4 +15,5 @@
   <xacro:arg name="use_lidar" default="true"/>
   <xacro:arg name="use_camera" default="true"/>
+  <xacro:arg name="camera_profile" default="$(find astribot_s1_description)/config/camera_generic.yaml"/>
   <!-- use_gripper：是否把平行夹爪作为真实关节模块建模。
        true（默认，与真机一致）：加载 astribot_s1_gripper.xacro，两臂末端各挂
@@ -45,5 +46,5 @@
        命名注意：URDF 沿用 left/right，实机话题叫 front/back，对应关系是
        **left = front = IP 192.168.0.12**，**right = back = IP 192.168.0.13**。
-       改名会牵动自滤配置、gazebo 传感器名与 livox_fusion_node，故本次只改数值。
+       改名会牵动自滤配置与 Gazebo 传感器名，故本次只改数值。
        坐标约定：torso_base 局部系 +x 朝前、+y 朝左。 -->
   <xacro:arg name="livox_left_xyz" default="0.17393 0.16893 0.082"/>
@@ -111,5 +112,5 @@
   </xacro:if>
   <xacro:if value="${use_camera_prop}">
-    <xacro:astribot_s1_camera parent="astribot_head_link_2" robot_name="${robot_name_prop}"/>
+    <xacro:astribot_s1_camera parent="astribot_head_link_2" robot_name="${robot_name_prop}" profile="$(arg camera_profile)"/>
   </xacro:if>
   <!-- ============ ros2_control + gz_ros2_control 插件 ============ -->

File: ws_robot/src/astribot_s1_description/urdf/astribot_s1_gripper.xacro (robot description, xacro)
@@ -127,25 +127,11 @@
   代价必须知道：**Gazebo 里这 6 个连杆的转动惯量被高估约 30 倍**，如果以后要在
   Gazebo 里做夹爪动力学（抓取力、指尖接触），这个值不能用。当前不用，故不改。
-  ================== Gazebo 侧 mimic：已实测，有 7.8° 稳态误差 ==================
-  此前这里写的是"Humble 的 gz_ros2_control 对 URDF <mimic> 的支持情况未实测，
-  从动关节可能受重力自由摆动"。**已实测（2026-08-20），结论是支持但不精确。**
-  测法：接 Gazebo 起全栈，给主动关节 joint_L1 下发 0.93 rad 并确认到位，
-  然后拿 Gazebo 内部的连杆位姿（ign topic /world/default/pose/info）
-  与 TF（robot_state_publisher 按 mimic 算出来的）逐个比。
-    astribot_gripper_left_Link_L11   Gazebo 与 TF 差 0.21 mm  —— 一致
-    astribot_gripper_left_Link_R11   Gazebo 与 TF 差 7.47 mm  —— 不一致
-  L11 的父关节是主动关节 L1（Gazebo 里真的被驱动），所以一致；
-  R11 的父关节 R1 是 mimic 关节。用 R11 的实测位置反解 R1 的真实角度：
-    R1(Gazebo) = 0.7940 rad，而 mimic 应给 0.9300 rad，
-    差 -0.1360 rad = **-7.79°**（反解残差 0.21 mm，解是干净的）。
-  注意 0.794 既不是 0（那会差 42.5 mm）也不是自由摆动的随机值 ——
-  所以 gz_ros2_control 确实在执行 mimic，只是像个有限刚度/带稳态误差的约束。
-  影响范围要分清：
-    · MoveIt 侧（规划与碰撞）用自己的 RobotState，mimic 是精确的，与厂商模型一致 ——
-      **规划结果不受影响**。
-    · Gazebo 侧的右指比 MoveIt 认为的少闭合约 15%。只要不依赖 Gazebo 的接触物理
-      做抓取（当前 transport 场景没有夹取/attach 动作），这个差异不进入结论。
-    · 一旦要用 Gazebo 做夹持力/接触实验，这 7.8° 必须先解决，
-      否则两指不对称、接触点也不对。
+  ================== Gazebo 侧 mimic ==================
+  URDF mimic只描述运动学关系，不能单凭从动连杆靠近理论位置认定物理耦合已生效。
+  2026-09-19复核：旧ros2_control仅声明L1，Gazebo日志没有加载其余五个从动关节；
+  实跑记录到从动杆与工位接触并触发机械臂跟踪保护。现于Gazebo ros2_control配置
+  显式声明从动关节的mimic/multiplier及状态接口，不建立独立控制器或command接口。
+  必须以加载日志、实际关节/连杆几何和接触记录验收，不能只检查TF。
+  仿真夹持仍为运动学附着，未证明夹持力、摩擦或滑落性能。
   ================== 本阶段（模型对齐）不做什么 ==================
   · 不做夹持力。厂商的夹持力是另一条接口（set_effector_max_force，10~80 N，

File: ws_robot/src/astribot_s1_description/urdf/astribot_s1_ros2_control.xacro (robot description, xacro)
@@ -25,4 +25,21 @@
       <state_interface name="velocity"/>
       <state_interface name="effort"/>
+    </joint>
+  </xacro:macro>
+  <!-- Only the master has a controller command interface. Humble's Gazebo
+       adapter requires explicit mimic parameters on the follower entries. -->
+  <xacro:macro name="astribot_s1_gripper_sim_mimics" params="side">
+    <xacro:astribot_s1_sim_mimic_joint side="${side}" suffix="L11" ratio="1"/>
+    <xacro:astribot_s1_sim_mimic_joint side="${side}" suffix="L2" ratio="-1"/>
+    <xacro:astribot_s1_sim_mimic_joint side="${side}" suffix="R1" ratio="1"/>
+    <xacro:astribot_s1_sim_mimic_joint side="${side}" suffix="R11" ratio="-1"/>
+    <xacro:astribot_s1_sim_mimic_joint side="${side}" suffix="R2" ratio="1"/>
+  </xacro:macro>
+  <xacro:macro name="astribot_s1_sim_mimic_joint" params="side suffix ratio">
+    <joint name="astribot_gripper_${side}_joint_${suffix}">
+      <param name="mimic">astribot_gripper_${side}_joint_L1</param>
+      <param name="multiplier">${ratio}</param>
+      <state_interface name="position"/>
+      <state_interface name="velocity"/>
     </joint>
   </xacro:macro>
@@ -82,18 +99,11 @@
       <xacro:astribot_s1_effort_wheel_joint name="wheel_RR_Joint"/>
       <xacro:astribot_s1_effort_wheel_joint name="wheel_LR_Joint"/>
-      <!-- 夹爪：每侧只声明**主动关节** joint_L1。
-           另外 5 个是 URDF mimic 关节，它们的位置由 robot_state_publisher 从主动
-           关节算出，既不该有 command_interface，也不该进 /joint_states ——
-           声明了反而会出现"同一个自由度被下发两次"。
-           !!! 不声明会怎样（实测）!!!
-           只把夹爪加进 URDF、不加到这里，move_group 会一直刷：
-             The complete state of the robot is not yet known.
-             Missing astribot_gripper_left_joint_L1, astribot_gripper_right_joint_L1
-           **拿不到完整机器人状态 => 规划完全不可用**。也就是说加夹爪这件事一旦
-           只做了模型那一半，现有的所有手臂 demo 会全部停摆，且报错信息指向
-           "状态未知"而不是"你漏配了控制器"，很容易查错方向。 -->
+      <!-- 主动关节由夹爪控制器驱动；从动关节仅交给Gazebo适配器的mimic
+           支路，不导出独立command interface。URDF mimic仍供MoveIt/TF使用。 -->
       <xacro:if value="${use_gripper}">
         <xacro:astribot_s1_position_joint name="astribot_gripper_left_joint_L1"/>
         <xacro:astribot_s1_position_joint name="astribot_gripper_right_joint_L1"/>
+        <xacro:astribot_s1_gripper_sim_mimics side="left"/>
+        <xacro:astribot_s1_gripper_sim_mimics side="right"/>
       </xacro:if>
     </ros2_control>

File: ws_robot/src/astribot_s1_description/urdf/astribot_s1_sensors.xacro (robot description, xacro)
@@ -53,5 +53,5 @@
          **都是** `livox_frame`（实测，直接解 CDR 取的）。而 TF 树里从来没有
          这个 frame —— 结果是任何靠 TF 摆放点云的消费者
-         （pointcloud_slice_scan_node 的自滤、livox_fusion_node）在实机上
+         （pointcloud_slice_scan_node 的自滤）在实机上
          直接查不到变换，而不是"位置略有偏差"。
          两路共用一个 frame_id 并**不是**厂商的疏漏：驱动通过
@@ -109,7 +109,20 @@
         </lidar>
       </sensor>
+      <!-- Voxel-SLAM consumes the same standard sensor_msgs/Imu topic in
+           simulation and on hardware.  Only the left/front sensor carries
+           the IMU so the two lidar streams do not create duplicate IMU
+           publishers. -->
+      <xacro:if value="${side == 'left'}">
+        <sensor name="livox_mid360_imu" type="imu">
+          <topic>/model/${robot_name}/livox_mid360_imu</topic>
+          <always_on>true</always_on>
+          <update_rate>200</update_rate>
+          <visualize>false</visualize>
+        </sensor>
+      </xacro:if>
     </gazebo>
   </xacro:macro>
-  <xacro:macro name="astribot_s1_camera" params="parent:=astribot_head_link_2 robot_name:=astribot_s1">
+  <xacro:macro name="astribot_s1_camera" params="parent:=astribot_head_link_2 robot_name:=astribot_s1 profile">
+    <xacro:property name="camera" value="${xacro.load_yaml(profile)}"/>
     <link name="camera_link">
       <inertial>
@@ -136,23 +149,28 @@
       <parent link="${parent}"/>
       <child link="camera_link"/>
-      <origin xyz="0 -0.22 0" rpy="-1.5708 0 -1.5708"/>
+      <origin xyz="${camera.mount_xyz}" rpy="${camera.mount_rpy}"/>
+    </joint>
+    <link name="camera_optical_frame"/>
+    <joint name="camera_optical_joint" type="fixed">
+      <parent link="camera_link"/><child link="camera_optical_frame"/>
+      <origin xyz="0 0 0" rpy="-1.5707963267948966 0 -1.5707963267948966"/>
     </joint>
     <gazebo reference="camera_link">
-      <sensor name="astribot_camera" type="camera">
+      <sensor name="astribot_camera" type="${camera.sensor_type}">
         <pose>0 0 0 0 0 0</pose>
-        <topic>/model/${robot_name}/camera/image_raw</topic>
-        <update_rate>30</update_rate>
+        <topic>${'/model/' + robot_name + '/camera' if camera.sensor_type == 'rgbd_camera' else '/model/' + robot_name + '/camera/image_raw'}</topic>
+        <update_rate>${camera.rate_hz}</update_rate>
         <always_on>true</always_on>
         <visualize>false</visualize>
         <camera>
-          <horizontal_fov>1.047</horizontal_fov>
+          <horizontal_fov>${camera.horizontal_fov}</horizontal_fov>
           <image>
-            <width>640</width>
-            <height>480</height>
+            <width>${camera.width}</width>
+            <height>${camera.height}</height>
             <format>R8G8B8</format>
           </image>
           <clip>
-            <near>0.05</near>
-            <far>50</far>
+            <near>${camera.near_m}</near>
+            <far>${camera.far_m}</far>
           </clip>
         </camera>
